File: 5BandCWTranceiver/main_1.kicad_sch (KiCad schematic)
At the start: 54 parts, among them J1 USB_B_Micro, J2 Conn_01x12_Female, J3 Conn_01x04_Female, J4 Conn_01x04_Female, J5 Conn_01x04_Female, J6 Conn_01x03_Female, U1 FT230XS, Y1 32.768kHz

Commit message: Update
Committing pcb/schematic updates
Parts:
- R2: value 39k -> 100
Changed lines of the file:
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@@
       (effects (font (size 1.778 1.5113)) (justify left bottom))
     )
-    (property "Value" "39k" (id 1) (at 95.25 53.34 90)
+    (property "Value" "100" (id 1) (at 95.25 53.34 90)
       (effects (font (size 1.778 1.5113)) (justify left bottom))
     )
