File: 5BandCWTranceiver/main_2.kicad_sch (KiCad schematic)
At the start: 59 parts, among them J10 Conn_01x02_Female, J11 Conn_01x02_Female, J12 Conn_01x02_Female, J13 Conn_01x04_Female, J14 Conn_01x02_Female, J15 Conn_01x02_Female, J16 Conn_01x02_Female, J17 Conn_01x02_Female, J18 Conn_01x02_Female, J19 Conn_01x02_Female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

Commit message: Update
Committing pcb/schematic updates
Parts:
- R23: value 1K -> 9.09K
- R38: value 39K -> 0
Other:
- note added: "Sideband Select"
Changed lines of the file:
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@@
     (stroke (width 0) (type default) (color 0 0 0 0))
+  )
+  (text "Sideband\nSelect" (at 191.77 57.15 0)
+    (effects (font (size 1.27 1.27)) (justify left bottom))
   )
   (text "to encoder switch" (at 19.05 191.77 180)
@@
     )
   )
-  (global_label "TUNER_ENCODER_SW" (shape bidirectional) (at 182.88 170.18 180) (fields_autoplaced)
-    (effects (font (size 1.2446 1.2446)) (justify right))
-    (property "Intersheet References" "${INTERSHEET_REFS}" (id 0) (at 327.66 -35.56 0)
+  (global_label "TUNER_ENCODER_SW" (shape bidirectional) (at 182.88 170.18 0) (fields_autoplaced)
+    (effects (font (size 1.2446 1.2446)) (justify left))
+    (property "Intersheet References" "${INTERSHEET_REFS}" (id 0) (at 38.1 375.92 0)
       (effects (font (size 1.27 1.27)) hide)
     )
@@
       (effects (font (size 1.778 1.5113)) (justify left bottom))
     )
-    (property "Value" "39K" (id 1) (at 251.46 59.69 0)
+    (property "Value" "0" (id 1) (at 251.46 59.69 0)
       (effects (font (size 1.778 1.5113)) (justify left bottom))
     )
@@
       (effects (font (size 1.778 1.5113)) (justify left bottom))
     )
-    (property "Value" "1K" (id 1) (at 40.64 76.2 90)
-      (effects (font (size 1.778 1.5113)) (justify left bottom))
-    )
+    (property "Value" "9.09K" (id 1) (at 38.1 77.47 90)
+      (effects (font (size 1.778 1.5113)) (justify left bottom))
+    )
