File: 5BandCWTranceiver/cwaz_lpf/cwaz_lpf.kicad_pcb (KiCad board)
At the start: 2 copper layers, 68.2 x 113 mm, 80 parts, among them J1 Conn_01x06_Male, J2 Conn_01x02_Male, J3 Conn_Coaxial, J4 Conn_Coaxial, J5 Conn_01x02_Male, J6 Conn_01x02_Male, J7 Conn_01x02_Male, J8 Conn_01x02_Male, J9 Conn_Coaxial, K1 G5V-2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

Commit message: Corrected LPF; add Preselector
Fixed circuit design error on LPF regarding relay connections; first pass at adding preselctor schematic
Parts:
- moved J9 0.50 mm to (93.6, 150.4)
- moved J4 0.50 mm to (103.6, 42.6)
- moved J3 0.50 mm to (108.4, 150.4)
Connections:
- C22 pad 1: Net-(C22-Pad1) -> Net-(K4-Pad4)
- C31 pad 1: Net-(C31-Pad1) -> Net-(K5-Pad13)
- C4 pad 1: Net-(C4-Pad1) -> Net-(K1-Pad4)
- J3 pad 1: Net-(J3-Pad1) -> Net-(K2-Pad8)
- J4 pad 1: Net-(J4-Pad1) -> Net-(K2-Pad9)
- J9 pad 1: Net-(J3-Pad1) -> Net-(K2-Pad8)
- K1 pad 13: Net-(J4-Pad1) -> Net-(C16-Pad1)
- K1 pad 4: Net-(J3-Pad1) -> Net-(K1-Pad4)
- K1 pad 8: Net-(C4-Pad1) -> Net-(K2-Pad8)
- K1 pad 9: Net-(C16-Pad1) -> Net-(K2-Pad9)
- K2 pad 13: Net-(J4-Pad1) -> Net-(C17-Pad1)
- K2 pad 4: Net-(J3-Pad1) -> Net-(C5-Pad1)
- K2 pad 8: Net-(C5-Pad1) -> Net-(K2-Pad8)
- K2 pad 9: Net-(C17-Pad1) -> Net-(K2-Pad9)
- K3 pad 13: Net-(J4-Pad1) -> Net-(C18-Pad1)
- K3 pad 4: Net-(J3-Pad1) -> Net-(C6-Pad1)
- K3 pad 8: Net-(C6-Pad1) -> Net-(K2-Pad8)
- K3 pad 9: Net-(C18-Pad1) -> Net-(K2-Pad9)
- K4 pad 13: Net-(J4-Pad1) -> Net-(C30-Pad1)
- K4 pad 4: Net-(J3-Pad1) -> Net-(K4-Pad4)
- K4 pad 8: Net-(C22-Pad1) -> Net-(K2-Pad8)
- K4 pad 9: Net-(C30-Pad1) -> Net-(K2-Pad9)
- K5 pad 13: Net-(J4-Pad1) -> Net-(K5-Pad13)
- K5 pad 4: Net-(J3-Pad1) -> Net-(C23-Pad1)
- K5 pad 8: Net-(C23-Pad1) -> Net-(K2-Pad8)
- K5 pad 9: Net-(C31-Pad1) -> Net-(K2-Pad9)
- L1 pad 2: Net-(C4-Pad1) -> Net-(K1-Pad4)
- L10 pad 2: Net-(C22-Pad1) -> Net-(K4-Pad4)
- L15 pad 1: Net-(C31-Pad1) -> Net-(K5-Pad13)
Routing:
- net Net-(K2-Pad8): track 0.00 -> 192.6 mm
- net Net-(K2-Pad9): track 0.00 -> 159.8 mm
- net Net-(J3-Pad1): track 122.3 -> 0.00 mm
- net Net-(J4-Pad1): track 112.9 -> 0.00 mm
- net Net-(K5-Pad13): track 0.00 -> 25.4 mm
- net Net-(K4-Pad4): track 0.00 -> 23.0 mm
- net Net-(K1-Pad4): track 0.00 -> 22.5 mm
- net Net-(C23-Pad1): track 13.6 -> 31.3 mm
- net Net-(C31-Pad1): track 15.1 -> 0.00 mm
- net Net-(C22-Pad1): track 14.6 -> 0.00 mm
- net Net-(C16-Pad1): track 15.1 -> 29.5 mm
- net Net-(C4-Pad1): track 14.2 -> 0.00 mm
- net Net-(C5-Pad1): track 13.8 -> 25.2 mm
- net Net-(C30-Pad1): track 14.9 -> 25.4 mm
- net Net-(C18-Pad1): track 14.9 -> 25.3 mm
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