File: 5BandCWTranceiver/cwaz_lpf/cwaz_lpf.kicad_sch (KiCad schematic)
At the start: 80 parts, among them J1 Conn_01x06_Male, J2 Conn_01x02_Male, J3 Conn_Coaxial, J4 Conn_Coaxial, J5 Conn_01x02_Male, J6 Conn_01x02_Male, J7 Conn_01x02_Male, J8 Conn_01x02_Male, J9 Conn_Coaxial, K1 G5V-2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

Commit message: Added T/R Switch
Added T/R switch and updated preselector.
Parts:
- R1, R2, R3, R7, R8: value R_US -> 2K
- R10, R4, R5, R6, R9: value R_US -> 3K
Other:
- note added: "Filter design based on QST Feb. 1999 article "Second-Harmonic-Optimized Low-Pass Filters" by Ed Wetherhold, W3NQN"
Changed lines of the file:
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@@
+    (effects (font (size 1.27 1.27)) (justify left bottom))
+  )
+  (text "Filter design based on QST Feb. 1999 article\n\"Second-Harmonic-Optimized Low-Pass Filters\" by\nEd Wetherhold, W3NQN"
+    (at 184.15 176.53 0)
     (effects (font (size 1.27 1.27)) (justify left bottom))
   )
@@
     (in_bom yes) (on_board yes) (fields_autoplaced)
     (property "Reference" "R1" (id 0) (at 41.91 29.21 90))
-    (property "Value" "R_US" (id 1) (at 41.91 31.75 90))
+    (property "Value" "2K" (id 1) (at 41.91 31.75 90))
     (property "Footprint" "Resistor_SMD:R_0603_1608Metric_Pad0.98x0.95mm_HandSolder" (id 2) (at 41.656 34.544 90)
       (effects (font (size 1.27 1.27)) hide)
@@
     (in_bom yes) (on_board yes) (fields_autoplaced)
     (property "Reference" "R8" (id 0) (at 167.64 85.09 90))
-    (property "Value" "R_US" (id 1) (at 167.64 87.63 90))
+    (property "Value" "2K" (id 1) (at 167.64 87.63 90))
     (property "Footprint" "Resistor_SMD:R_0603_1608Metric_Pad0.98x0.95mm_HandSolder" (id 2) (at 167.386 90.424 90)
       (effects (font (size 1.27 1.27)) hide)
@@
   (symbol (lib_id "Device:R_US") (at 48.26 92.71 0) (mirror y) (unit 1)
     (in_bom yes) (on_board yes) (fields_autoplaced)
-    (property "Reference" "R5" (id 0) (at 45.72 91.4399 0)
-      (effects (font (size 1.27 1.27)) (justify left))
-    )
-    (property "Value" "R_US" (id 1) (at 45.72 93.9799 0)
-      (effects (font (size 1.27 1.27)) (justify left))
+    (property "Reference" "R5" (id 0) (at 50.8 91.4399 0)
+      (effects (font (size 1.27 1.27)) (justify right))
+    )
+    (property "Value" "3K" (id 1) (at 50.8 93.9799 0)
+      (effects (font (size 1.27 1.27)) (justify right))
     )
     (property "Footprint" "Resistor_SMD:R_0603_1608Metric_Pad0.98x0.95mm_HandSolder" (id 2) (at 47.244 92.964 90)
@@
     (in_bom yes) (on_board yes) (fields_autoplaced)
     (property "Reference" "R7" (id 0) (at 167.64 29.21 90))
-    (property "Value" "R_US" (id 1) (at 167.64 31.75 90))
+    (property "Value" "2K" (id 1) (at 167.64 31.75 90))
     (property "Footprint" "Resistor_SMD:R_0603_1608Metric_Pad0.98x0.95mm_HandSolder" (id 2) (at 167.386 34.544 90)
       (effects (font (size 1.27 1.27)) hide)
@@
   (symbol (lib_id "Device:R_US") (at 48.26 48.26 0) (mirror y) (unit 1)
     (in_bom yes) (on_board yes) (fields_autoplaced)
-    (property "Reference" "R4" (id 0) (at 45.72 46.9899 0)
-      (effects (font (size 1.27 1.27)) (justify left))
-    )
-    (property "Value" "R_US" (id 1) (at 45.72 49.5299 0)
-      (effects (font (size 1.27 1.27)) (justify left))
+    (property "Reference" "R4" (id 0) (at 50.8 46.9899 0)
+      (effects (font (size 1.27 1.27)) (justify right))
+    )
+    (property "Value" "3K" (id 1) (at 50.8 49.5299 0)
+      (effects (font (size 1.27 1.27)) (justify right))
     )
     (property "Footprint" "Resistor_SMD:R_0603_1608Metric_Pad0.98x0.95mm_HandSolder" (id 2) (at 47.244 48.514 90)
@@
   (symbol (lib_id "Device:R_US") (at 173.99 104.14 0) (mirror y) (unit 1)
     (in_bom yes) (on_board yes) (fields_autoplaced)
-    (property "Reference" "R10" (id 0) (at 171.45 102.8699 0)
-      (effects (font (size 1.27 1.27)) (justify left))
-    )
-    (property "Value" "R_US" (id 1) (at 171.45 105.4099 0)
-      (effects (font (size 1.27 1.27)) (justify left))
+    (property "Reference" "R10" (id 0) (at 176.53 102.8699 0)
+      (effects (font (size 1.27 1.27)) (justify right))
+    )
+    (property "Value" "3K" (id 1) (at 176.53 105.4099 0)
+      (effects (font (size 1.27 1.27)) (justify right))
     )
     (property "Footprint" "Resistor_SMD:R_0603_1608Metric_Pad0.98x0.95mm_HandSolder" (id 2) (at 172.974 104.394 90)
@@
     (in_bom yes) (on_board yes) (fields_autoplaced)
     (property "Reference" "R3" (id 0) (at 41.91 120.65 90))
-    (property "Value" "R_US" (id 1) (at 41.91 123.19 90))
+    (property "Value" "2K" (id 1) (at 41.91 123.19 90))
     (property "Footprint" "Resistor_SMD:R_0603_1608Metric_Pad0.98x0.95mm_HandSolder" (id 2) (at 41.656 125.984 90)
       (effects (font (size 1.27 1.27)) hide)
@@
   (symbol (lib_id "Device:R_US") (at 48.26 139.7 0) (mirror y) (unit 1)
     (in_bom yes) (on_board yes) (fields_autoplaced)
-    (property "Reference" "R6" (id 0) (at 45.72 138.4299 0)
-      (effects (font (size 1.27 1.27)) (justify left))
-    )
-    (property "Value" "R_US" (id 1) (at 45.72 140.9699 0)
-      (effects (font (size 1.27 1.27)) (justify left))
+    (property "Reference" "R6" (id 0) (at 50.8 138.4299 0)
+      (effects (font (size 1.27 1.27)) (justify right))
+    )
+    (property "Value" "3K" (id 1) (at 50.8 140.9699 0)
+      (effects (font (size 1.27 1.27)) (justify right))
     )
     (property "Footprint" "Resistor_SMD:R_0603_1608Metric_Pad0.98x0.95mm_HandSolder" (id 2) (at 47.244 139.954 90)
@@
     (in_bom yes) (on_board yes) (fields_autoplaced)
     (property "Reference" "R2" (id 0) (at 41.91 73.66 90))
-    (property "Value" "R_US" (id 1) (at 41.91 76.2 90))
+    (property "Value" "2K" (id 1) (at 41.91 76.2 90))
     (property "Footprint" "Resistor_SMD:R_0603_1608Metric_Pad0.98x0.95mm_HandSolder" (id 2) (at 41.656 78.994 90)
       (effects (font (size 1.27 1.27)) hide)
@@
   (symbol (lib_id "Device:R_US") (at 173.99 48.26 0) (mirror y) (unit 1)
     (in_bom yes) (on_board yes) (fields_autoplaced)
-    (property "Reference" "R9" (id 0) (at 171.45 46.9899 0)
-      (effects (font (size 1.27 1.27)) (justify left))
-    )
-    (property "Value" "R_US" (id 1) (at 171.45 49.5299 0)
-      (effects (font (size 1.27 1.27)) (justify left))
+    (property "Reference" "R9" (id 0) (at 176.53 46.9899 0)
+      (effects (font (size 1.27 1.27)) (justify right))
+    )
+    (property "Value" "3K" (id 1) (at 176.53 49.5299 0)
+      (effects (font (size 1.27 1.27)) (justify right))
     )
     (property "Footprint" "Resistor_SMD:R_0603_1608Metric_Pad0.98x0.95mm_HandSolder" (id 2) (at 172.974 48.514 90)
@@
     )
     (path "/506ae28c-26c6-4640-84e4-7bc0e7e07d3f"
-      (reference "R1") (unit 1) (value "R_US") (footprint "Resistor_SMD:R_0603_1608Metric_Pad0.98x0.95mm_HandSolder")
+      (reference "R1") (unit 1) (value "2K") (footprint "Resistor_SMD:R_0603_1608Metric_Pad0.98x0.95mm_HandSolder")
     )
     (path "/d97c1df9-afd6-4cd6-8b65-79ac20616477"
-      (reference "R2") (unit 1) (value "R_US") (footprint "Resistor_SMD:R_0603_1608Metric_Pad0.98x0.95mm_HandSolder")
+      (reference "R2") (unit 1) (value "2K") (footprint "Resistor_SMD:R_0603_1608Metric_Pad0.98x0.95mm_HandSolder")
     )
     (path "/c7c95ec0-d804-4c5a-b1c0-1db8cf595862"
-      (reference "R3") (unit 1) (value "R_US") (footprint "Resistor_SMD:R_0603_1608Metric_Pad0.98x0.95mm_HandSolder")
+      (reference "R3") (unit 1) (value "2K") (footprint "Resistor_SMD:R_0603_1608Metric_Pad0.98x0.95mm_HandSolder")
     )
     (path "/89c1603c-11e6-411d-b684-f66ff3e675f7"
-      (reference "R4") (unit 1) (value "R_US") (footprint "Resistor_SMD:R_0603_1608Metric_Pad0.98x0.95mm_HandSolder")
+      (reference "R4") (unit 1) (value "3K") (footprint "Resistor_SMD:R_0603_1608Metric_Pad0.98x0.95mm_HandSolder")
     )
     (path "/53c4130b-71fa-42d5-a7e1-a6817377c820"
-      (reference "R5") (unit 1) (value "R_US") (footprint "Resistor_SMD:R_0603_1608Metric_Pad0.98x0.95mm_HandSolder")
+      (reference "R5") (unit 1) (value "3K") (footprint "Resistor_SMD:R_0603_1608Metric_Pad0.98x0.95mm_HandSolder")
     )
     (path "/d9207482-0f82-4864-b4c1-997d17d34896"
-      (reference "R6") (unit 1) (value "R_US") (footprint "Resistor_SMD:R_0603_1608Metric_Pad0.98x0.95mm_HandSolder")
+      (reference "R6") (unit 1) (value "3K") (footprint "Resistor_SMD:R_0603_1608Metric_Pad0.98x0.95mm_HandSolder")
     )
     (path "/6f06a029-aa7a-422b-bb4c-cd92722acf24"
-      (reference "R7") (unit 1) (value "R_US") (footprint "Resistor_SMD:R_0603_1608Metric_Pad0.98x0.95mm_HandSolder")
+      (reference "R7") (unit 1) (value "2K") (footprint "Resistor_SMD:R_0603_1608Metric_Pad0.98x0.95mm_HandSolder")
     )
     (path "/51a6d19c-f5c6-4812-b125-1223119ed67a"
-      (reference "R8") (unit 1) (value "R_US") (footprint "Resistor_SMD:R_0603_1608Metric_Pad0.98x0.95mm_HandSolder")
+      (reference "R8") (unit 1) (value "2K") (footprint "Resistor_SMD:R_0603_1608Metric_Pad0.98x0.95mm_HandSolder")
     )
     (path "/fbeabe29-b707-4505-ba93-3240ae9fe773"
-      (reference "R9") (unit 1) (value "R_US") (footprint "Resistor_SMD:R_0603_1608Metric_Pad0.98x0.95mm_HandSolder")
+      (reference "R9") (unit 1) (value "3K") (footprint "Resistor_SMD:R_0603_1608Metric_Pad0.98x0.95mm_HandSolder")
     )
     (path "/ae6f726f-79a6-45eb-8c95-2c6f0edd887c"
-      (reference "R10") (unit 1) (value "R_US") (footprint "Resistor_SMD:R_0603_1608Metric_Pad0.98x0.95mm_HandSolder")
-    )
-  )
+      (reference "R10") (unit 1) (value "3K") (footprint "Resistor_SMD:R_0603_1608Metric_Pad0.98x0.95mm_HandSolder")
+    )
+  )
