File: 5BandCWTranceiver/qsd/qsd_revB.kicad_pcb (KiCad board)
At the start: 2 copper layers, 55.9 x 37.1 mm, 56 parts, among them IC1 MCP1801, IC2 SN74LVC1G04DBVT, IC3 SN74AUP2G79DCUR, IC4 TS5A23157, IC5 SN74CBTLV3253, IC6 SN74LVC1G04DBVT, J1 Conn_Coaxial, J2 Conn_Coaxial, J3 Conn_Coaxial, Q1 J309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

Commit message: Tape Out of T/RBoard and QSD
Rev. B of T/R board and Rev. C of Tayloe detector board
Parts:
- C1, C11, C4: footprint qsd_revB:0603-CAP -> Capacitor_SMD:C_0603_1608Metric_Pad1.08x0.95mm_HandSolder
Routing:
- net GND: vias 38 -> 41
