File: 5BandCWTranceiver/audioFilters/audioFilters.kicad_pcb (KiCad board)
At the start: 2 copper layers, 73 x 45.8 mm, 102 parts, among them J1 Conn_01x02, J2 Conn_01x03, J3 Conn_01x02, J4 Conn_01x02, J5 Conn_01x02, J6 Conn_01x02, U1 OPA1678, U2 OPA1678, U3 OPA1678, U4 OPA1678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

Commit message: First Pass Routing
first pass routing of audio filter board
Parts:
- moved C1 15.6 mm to (153.0, 79.6), turned to 180 degrees
- moved C9 14.3 mm to (172.8, 87.0)
- moved R46 2.06 mm to (158.8, 111.8)
- moved C37 1.94 mm to (158.8, 113.8)
- moved R8 0.12 mm to (123.6, 95.5)
Routing:
- net VCC5: track 0.00 -> 165.2 mm, vias 0 -> 5
- net Net-(R24-Pad1): track 0.00 -> 78.1 mm, vias 0 -> 2
- net VBIAS: track 0.00 -> 64.2 mm, vias 0 -> 3
- net Net-(C36-Pad1): track 0.00 -> 22.5 mm
- net Net-(J2-Pad1): track 0.00 -> 21.6 mm
- net Net-(C8-Pad1): track 0.00 -> 21.2 mm
- net allPass_out: track 0.00 -> 20.6 mm
- net Net-(R10-Pad1): track 0.00 -> 19.5 mm
- net Net-(C23-Pad1): track 0.00 -> 19.4 mm
- net Net-(C20-Pad2): track 0.00 -> 19.3 mm
- net Net-(C19-Pad2): track 0.00 -> 19.2 mm
- net Net-(C35-Pad2): track 0.00 -> 17.5 mm, vias 0 -> 2
- net Net-(R14-Pad2): track 0.00 -> 17.3 mm
- net Net-(C34-Pad2): track 0.00 -> 16.8 mm, vias 0 -> 2
- net Net-(R15-Pad2): track 0.00 -> 15.8 mm
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- added copper zone on B.Cu, net GND
- added copper zone on F.Cu, net GND

Commit message: audioFilters board tapeout
ready for tapeout
Parts:
- added J10: Conn_01x02, Connector_PinHeader_2.54mm:PinHeader_1x02_P2.54mm_Vertical, F.Cu at (125.1, 119.8)
- added J7: Conn_01x02, Connector_PinHeader_2.54mm:PinHeader_1x02_P2.54mm_Vertical, F.Cu at (108.2, 81.5)
- added J8: Conn_01x02, Connector_PinHeader_2.54mm:PinHeader_1x02_P2.54mm_Vertical, F.Cu at (170.7, 119.8)
- added J9: Conn_01x02, Connector_PinHeader_2.54mm:PinHeader_1x02_P2.54mm_Vertical, F.Cu at (171.8, 79.6)
Routing:
- net GND: vias 47 -> 45
Other:
- board text added: "AllPass Audio Filters N7WMN Rev. A"
- board text added: "GND"
- board text added: "I"
- board text added: "NARROW"
- board text added: "Q"
- board text added: "VBIAS"
- board text added: "VCC5"
- board text added: "WIDE"
- board text added: "allpass out"
