File: 5BandCWTranceiver/audioFilters/hplp_filters.kicad_sch (KiCad schematic)
At the start: 0 parts

Commit message: Start allpass+filters
Initial commit of board combining allpass and hp, lp filters
Parts:
- added C? (x5): 0.012uF, Capacitor_SMD:C_0603_1608Metric_Pad1.08x0.95mm_HandSolder, symbol Device:C
- added C? (x4): 0.0033uF, Capacitor_SMD:C_0603_1608Metric_Pad1.08x0.95mm_HandSolder, symbol Device:C
- added C?: 0.0039uF, Capacitor_SMD:C_0603_1608Metric_Pad1.08x0.95mm_HandSolder, symbol Device:C
- added C?: 0.039uF, Capacitor_SMD:C_0603_1608Metric_Pad1.08x0.95mm_HandSolder, symbol Device:C
- added C?: 1uF, Capacitor_SMD:C_0603_1608Metric_Pad1.08x0.95mm_HandSolder, symbol Device:C
- added C? (x2): 0.47uF, Capacitor_SMD:C_0603_1608Metric_Pad1.08x0.95mm_HandSolder, symbol Device:C
- added C? (x4): 0.1uF, Capacitor_SMD:C_0603_1608Metric_Pad1.08x0.95mm_HandSolder, symbol Device:C
- added C?: 0.39uF, Capacitor_SMD:C_0603_1608Metric_Pad1.08x0.95mm_HandSolder, symbol Device:C
- added C?: 0.018uF, Capacitor_SMD:C_0603_1608Metric_Pad1.08x0.95mm_HandSolder, symbol Device:C
- added C?: 0.82uF, Capacitor_SMD:C_0603_1608Metric_Pad1.08x0.95mm_HandSolder, symbol Device:C
- added C?: 0.22uF, Capacitor_SMD:C_0603_1608Metric_Pad1.08x0.95mm_HandSolder, symbol Device:C
- added C?: 1.5uF, Capacitor_SMD:C_0603_1608Metric_Pad1.08x0.95mm_HandSolder, symbol Device:C
- added C?: 0.33uF, Capacitor_SMD:C_0603_1608Metric_Pad1.08x0.95mm_HandSolder, symbol Device:C
- added C?: 0.0056uF, Capacitor_SMD:C_0603_1608Metric_Pad1.08x0.95mm_HandSolder, symbol Device:C
- added C?: 0.015uF, Capacitor_SMD:C_0603_1608Metric_Pad1.08x0.95mm_HandSolder, symbol Device:C
- added C?: 0.68uF, Capacitor_SMD:C_0603_1608Metric_Pad1.08x0.95mm_HandSolder, symbol Device:C
- added R?: 4.32K, Resistor_SMD:R_0603_1608Metric_Pad0.98x0.95mm_HandSolder, symbol Device:R_US
- added R?: 8.06K, Resistor_SMD:R_0603_1608Metric_Pad0.98x0.95mm_HandSolder, symbol Device:R_US
- added R?: 8.66K, Resistor_SMD:R_0603_1608Metric_Pad0.98x0.95mm_HandSolder, symbol Device:R_US
- added R?: 1K, Resistor_SMD:R_0603_1608Metric_Pad0.98x0.95mm_HandSolder, symbol Device:R_US
- added R?: 10.5K, Resistor_SMD:R_0603_1608Metric_Pad0.98x0.95mm_HandSolder, symbol Device:R_US
- added R?: 9.76K, Resistor_SMD:R_0603_1608Metric_Pad0.98x0.95mm_HandSolder, symbol Device:R_US
- added R?: 604, Resistor_SMD:R_0603_1608Metric_Pad0.98x0.95mm_HandSolder, symbol Device:R_US
- added R?: 3.92K, Resistor_SMD:R_0603_1608Metric_Pad0.98x0.95mm_HandSolder, symbol Device:R_US
- added R?: 9.53K, Resistor_SMD:R_0603_1608Metric_Pad0.98x0.95mm_HandSolder, symbol Device:R_US
- added R? (x2): 1.02K, Resistor_SMD:R_0603_1608Metric_Pad0.98x0.95mm_HandSolder, symbol Device:R_US
- added R?: 18.7K, Resistor_SMD:R_0603_1608Metric_Pad0.98x0.95mm_HandSolder, symbol Device:R_US
- added R?: 267, Resistor_SMD:R_0603_1608Metric_Pad0.98x0.95mm_HandSolder, symbol Device:R_US
- added R?: 21K, Resistor_SMD:R_0603_1608Metric_Pad0.98x0.95mm_HandSolder, symbol Device:R_US
- added R?: 11.8K, Resistor_SMD:R_0603_1608Metric_Pad0.98x0.95mm_HandSolder, symbol Device:R_US
- added R?: 16.5K, Resistor_SMD:R_0603_1608Metric_Pad0.98x0.95mm_HandSolder, symbol Device:R_US
- added R?: 866, Resistor_SMD:R_0603_1608Metric_Pad0.98x0.95mm_HandSolder, symbol Device:R_US
- added R?: 2.55K, Resistor_SMD:R_0603_1608Metric_Pad0.98x0.95mm_HandSolder, symbol Device:R_US
- added R?: 1.96K, Resistor_SMD:R_0603_1608Metric_Pad0.98x0.95mm_HandSolder, symbol Device:R_US
- added R?: 11K, Resistor_SMD:R_0603_1608Metric_Pad0.98x0.95mm_HandSolder, symbol Device:R_US
- added R?: 9.09K, Resistor_SMD:R_0603_1608Metric_Pad0.98x0.95mm_HandSolder, symbol Device:R_US
- added R?: 23.2K, Resistor_SMD:R_0603_1608Metric_Pad0.98x0.95mm_HandSolder, symbol Device:R_US
- added R?: 301, Resistor_SMD:R_0603_1608Metric_Pad0.98x0.95mm_HandSolder, symbol Device:R_US
- added R?: 6.04K, Resistor_SMD:R_0603_1608Metric_Pad0.98x0.95mm_HandSolder, symbol Device:R_US
- added U? (x14): OPA1679, symbol Amplifier_Operational:OPA1679
- added U?: OPA1679, Package_SO:SOIC-14_3.9x8.7mm_P1.27mm, symbol Amplifier_Operational:OPA1679
Connections:
- new net: C?.1, R?.2, U?.5 (+) (x2)
- new net: C?.1, R?.1, R?.2 (x8)
- new net: C?.2, R?.1, U?.1, U?.2 (-) (x2)
- new net: C?.2, R?.2, U?.10 (+)
- new net: C?.1, R?.2, U?.8, U?.9 (-)
- new net: C?.2, R?.1, U?.13 (-), U?.14 (x2)
- new net: C?.1, R?.2, U?.12 (+) (x2)
- new net: C?.2, R?.2, U?.12 (+)
- new net: R?.1, R?.1, R?.2, U?.6 (-), U?.7
- new net: C?.2, R?.1, U?.8, U?.9 (-) (x2)
- new net: C?.1, R?.2, U?.10 (+) (x2)
- new net: C?.1, C?.2, R?.1 (x4)
- new net: C?.1, R?.2, U?.13 (-), U?.14
- new net: C?.1, R?.2, U?.1, U?.2 (-)
- new net: C?.1, R?.2, U?.3 (+) (x2)
- new net: C?.2, R?.2, U?.3 (+)
- new net: C?.2, R?.2, U?.5 (+)
- new net GND: C?.1, C?.1, C?.1, C?.2, C?.2, C?.2, C?.2, C?.2, C?.2, C?.2, C?.2, U?.11 (V-), U?.11 (V-), U?.11 (V-)
- new net NARROW: C?.2, U?.6 (-), U?.7
- new net VBIAS: R?.1, R?.1, R?.1, R?.1
- new net VCC5: C?.2, C?.2, C?.2, U?.4 (V+), U?.4 (V+), U?.4 (V+)
- new net WIDE: C?.2, U?.6 (-), U?.7
- new net allPass_out: C?.1
Other:
- note added: "300 Hz High Pass"
- note added: "3kHz Low Pass"
- note added: "800 Hz Low Pass"

Commit message: Initial Placement
Initial placement of audio filter board
Parts:
- U5, U6, U7: renamed from U?; footprint (none) -> Package_SO:SOIC-14_3.9x8.7mm_P1.27mm
- gave numbers to parts that had none: 54
Other:
- note added: "All Pass Filter and Wide/Narrow Audio Filters"

Commit message: Field Radio First Pass
Starting assembly of field radio schematics
Connections:
- net NARROW renamed narrow
- net VBIAS renamed vbias
- net WIDE renamed wide
- net allPass_out renamed in
