File: 5BandCWTranceiver/audio/audioModule2.kicad_pcb (KiCad board)
At the start: 2 copper layers, 79.4 x 32.4 mm, 59 parts, among them Q1 MMBT3906, Q2 MMBT3904, Q3 PZT2222A, Q4 PZT2907A

Commit message: Update Audio Board
modify design and layout improvements
Parts:
- removed C8: 0.1uF, Capacitor_SMD:C_0603_1608Metric_Pad1.08x0.95mm_HandSolder
- added C17: 4.7uF, Capacitor_THT:CP_Radial_D6.3mm_P2.50mm, F.Cu at (105.8, 119.7)
- added C18: 0.1uF, Capacitor_SMD:C_0603_1608Metric_Pad1.08x0.95mm_HandSolder, F.Cu at (119.2, 119.3)
- added C19: 4.7uF, Capacitor_SMD:C_0603_1608Metric_Pad1.08x0.95mm_HandSolder, F.Cu at (122.7, 113.5)
- added JP14: VBIAS, Connector_PinHeader_2.54mm:PinHeader_1x02_P2.54mm_Vertical, F.Cu at (96.5, 127.1)
- C12: value 4.7uF -> 47uF
- C3: value CAP_POLPTH1 -> 4.7uF
- R10: value 100 -> 270
- R14: value 100 -> 604
- R16: value 15K -> 14.3k
- R17: value 68 -> 75
- R2, R3: moved to F.Cu
- R4: value 10K -> 22; footprint Resistor_SMD:R_0603_1608Metric_Pad0.98x0.95mm_HandSolder -> Resistor_SMD:R_0805_2012Metric_Pad1.20x1.40mm_HandSolder
- R8: value 33 -> 22; footprint Resistor_SMD:R_0603_1608Metric_Pad0.98x0.95mm_HandSolder -> Resistor_SMD:R_0805_2012Metric_Pad1.20x1.40mm_HandSolder
- RV2: value 5K -> 2K
- moved R8 50.2 mm to (142.4, 127.8), turned to 0 degrees
- moved C4 49.0 mm to (140.2, 104.5), turned to 180 degrees
- moved R4 46.1 mm to (142.2, 117.2), turned to 0 degrees
- moved JP1 43.0 mm to (138.9, 100.3), turned to 90 degrees
- moved C9 37.1 mm to (134.4, 101.1)
- moved C1 17.1 mm to (94.6, 106.3)
- moved JP7 7.99 mm to (124.7, 99.9)
- moved C14 7.07 mm to (109.2, 125.1), turned to -90 degrees
- moved JP3 4.01 mm to (103.1, 127.1)
- moved R15 3.79 mm to (122.4, 122.9), turned to 0 degrees
- moved JP10 2.64 mm to (88.7, 99.9)
- moved R16 1.66 mm to (133.6, 113.1)
- moved R2 0.85 mm to (83.4, 124.5)
Connections:
- C2 pad 1: Net-(C2-Pad1) -> /VBIAS
- C3 pad 1: Net-(C2-Pad1) -> /VBIAS
- C4 pad 2: Net-(C4-Pad2) -> /VCC12
- C9 pad 1: Net-(C8-Pad2) -> /VCC12
- D1 pad 2: Net-(C8-Pad2) -> /VCC12
- JP1 pad 1: Net-(C4-Pad2) -> /VCC12
- Q3 pad 1: Net-(Q1-Pad3) -> Net-(Q3-Pad1)
- Q3 pad 2: Net-(C8-Pad2) -> /VCC12
- Q3 pad 4: Net-(C8-Pad2) -> /VCC12
- Q4 pad 1: Net-(Q2-Pad2) -> Net-(Q4-Pad1)
- R1 pad 2: Net-(C2-Pad1) -> /VBIAS
- R12 pad 1: Net-(C8-Pad2) -> /VCC12
- R17 pad 1: Net-(C8-Pad2) -> /VCC12
- R4 pad 1: /VCC5 -> Net-(Q1-Pad3)
- R4 pad 2: Net-(C2-Pad1) -> Net-(Q3-Pad1)
- R5 pad 2: Net-(C4-Pad2) -> /VCC12
- R8 pad 1: Net-(C8-Pad2) -> Net-(Q2-Pad2)
- R8 pad 2: Net-(C4-Pad2) -> Net-(Q4-Pad1)
- U$1 pad 4: Net-(C2-Pad1) -> /VBIAS
- U$2 pad 8: Net-(C8-Pad2) -> /VCC12
Routing:
- net /VCC12: track 0.00 -> 97.2 mm, vias 0 -> 3
- net Net-(C8-Pad2): track 93.0 -> 0.00 mm, vias 2 -> 0
- net Net-(C4-Pad2): track 28.9 -> 0.00 mm, vias 1 -> 0
- net /VBIAS: track 0.00 -> 16.7 mm
- net Net-(C2-Pad1): track 13.6 -> 0.00 mm
- net Net-(C14-Pad2): track 10.9 -> 17.7 mm
- net Net-(Q1-Pad3): track 28.8 -> 22.7 mm
- net Net-(Q2-Pad2): track 43.7 -> 39.8 mm
- net Net-(Q3-Pad1): track 0.00 -> 3.79 mm
- net Net-(Q4-Pad1): track 0.00 -> 3.44 mm
- net /MUTE: track 18.6 -> 15.7 mm
- net Net-(D2-Pad1): track 8.04 -> 6.44 mm
- net Net-(C12-Pad1): track 30.2 -> 31.5 mm
- net Net-(JP11-Pad2): track 6.97 -> 7.76 mm
- net /VCC5: track 32.8 -> 33.5 mm
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Other:
- board text added: "N7WMN Audio Module 6"
- board text added: "VBIAS"
- board text removed: "N7WMN Audio Module 5"

Commit message: Tapeout - audio and power boards
Last mods to audio board; new power board
Parts:
- removed RV1: R_Potentiometer_US, Potentiometer_THT:Potentiometer_Bourns_3296W_Vertical
- added C8: 4.7uF, Capacitor_THT:CP_Radial_D6.3mm_P2.50mm, F.Cu at (104.0, 103.3)
- C12: value 47uF -> 4.7uF; footprint Capacitor_SMD:C_0603_1608Metric_Pad1.08x0.95mm_HandSolder -> Capacitor_THT:CP_Radial_D6.3mm_P2.50mm; moved to B.Cu
- R4, R8: value 22 -> 47
- U$2: value LM4562 -> OPA1678
- moved C12 25.6 mm to (134.2, 111.6), turned to -90 degrees
- moved R10 10.1 mm to (99.4, 110.7)
- moved Q1 2.99 mm to (127.2, 113.3)
- moved R14 2.92 mm to (113.2, 106.9)
- moved R8 2.81 mm to (139.6, 127.5)
- moved R16 2.61 mm to (131.0, 113.3)
- moved R17 1.02 mm to (133.8, 106.9)
- moved JP7 0.89 mm to (123.9, 100.1)
Connections:
- C12 pad 1: Net-(C12-Pad1) -> Net-(Q1-Pad3)
- C12 pad 2: Net-(C12-Pad2) -> Net-(Q2-Pad2)
- C15 pad 2: Net-(C12-Pad1) -> Net-(C15-Pad2)
- R10 pad 2: Net-(C12-Pad2) -> Net-(R10-Pad2)
- R14 pad 1: Net-(R14-Pad1) -> Net-(U$2-Pad1)
- R15 pad 1: Net-(C12-Pad1) -> Net-(C15-Pad2)
- U$2 pad 1: Net-(RV1-Pad1) -> Net-(U$2-Pad1)
- U$2 pad 2: Net-(RV1-Pad1) -> Net-(U$2-Pad1)
- U$2 pad 6: Net-(C12-Pad1) -> Net-(C15-Pad2)
Routing:
- net Net-(C15-Pad2): track 0.00 -> 34.8 mm
- net Net-(C12-Pad1): track 31.5 -> 0.00 mm
- net Net-(RV1-Pad1): track 14.4 -> 0.00 mm
- net Net-(U$2-Pad1): track 0.00 -> 14.2 mm
- net Net-(R10-Pad1): track 16.9 -> 7.75 mm
- net Net-(Q1-Pad3): track 22.7 -> 30.7 mm
- net Net-(R10-Pad2): track 0.00 -> 7.89 mm
- net Net-(Q2-Pad2): track 39.8 -> 46.5 mm, vias 1 -> 2
- net Net-(C12-Pad2): track 3.94 -> 0.00 mm
- net Net-(R14-Pad1): track 3.92 -> 0.00 mm
- net Net-(C16-Pad1): track 33.0 -> 35.4 mm
- net Net-(Q4-Pad1): track 3.44 -> 5.24 mm
- net Net-(Q1-Pad2): track 9.87 -> 10.4 mm
