File: 5BandCWTranceiver/optLowPass/optLowPass/optLowPass.kicad_sch (KiCad schematic)
At the start: 84 parts, among them J1 Conn_01x06_Male, J2 Conn_01x02_Male, J3 Conn_Coaxial, J4 Conn_Coaxial, J5 Conn_01x02_Male, J6 Conn_01x02_Male, J7 Conn_01x02_Male, J8 Conn_01x02_Male, Q1 BSS123, Q2 BSS123, Q3 BSS123, Q4 BSS123, Q5 BSS123

Commit message: Updating field radio
Continued schematic work on field radio
Parts:
- C10: value 202p -> 200p
- C12: value 101p -> 100p
- C13: value 557p -> 560p
- C15: value 279p -> 270p
- C18: value 44p -> 47p
- C23: value 209p -> 200p
- C27: value 67p -> 62p
- C28: value 217p -> 220p
- C32: value 628p -> 620p
- C33: value 89p -> 91p
- C34: value 1218p -> 1200p
- C37: value 435p -> 430p
- C39: value 844p -> 820p
- C40: value 140p -> 150p
- C41: value 386p -> 390p
- C44: value 609p -> 620p
- C47: value 244p -> 240p
- C48: value 35p -> 33p
- C49: value 474p -> 470p
- C50: value 79p -> 82p
- C53: value 30p -> 33p
- C54: value 406p -> 390p
- C56: value 186p -> 180p
- C6: value 314p -> 330p
Changed lines of the file:
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@@
       (effects (font (size 1.27 1.27)))
     )
-    (property "Value" "202p" (at 116.84 44.45 90)
+    (property "Value" "200p" (at 116.84 44.45 90)
       (effects (font (size 1.27 1.27)))
     )
@@
       (effects (font (size 1.27 1.27)) (justify left))
     )
-    (property "Value" "314p" (at 93.98 97.79 0)
+    (property "Value" "330p" (at 93.98 97.79 0)
       (effects (font (size 1.27 1.27)) (justify left))
     )
@@
       (effects (font (size 1.27 1.27)) (justify left))
     )
-    (property "Value" "186p" (at 130.81 154.94 0)
+    (property "Value" "180p" (at 130.81 154.94 0)
       (effects (font (size 1.27 1.27)) (justify left))
     )
@@
       (effects (font (size 1.27 1.27)) (justify left))
     )
-    (property "Value" "406p" (at 107.95 154.94 0)
+    (property "Value" "390p" (at 107.95 154.94 0)
       (effects (font (size 1.27 1.27)) (justify left))
     )
@@
       (effects (font (size 1.27 1.27)) (justify left))
     )
-    (property "Value" "244p" (at 93.98 123.19 0)
+    (property "Value" "240p" (at 93.98 123.19 0)
       (effects (font (size 1.27 1.27)) (justify left))
     )
@@
       (effects (font (size 1.27 1.27)))
     )
-    (property "Value" "140p" (at 118.11 71.12 90)
+    (property "Value" "150p" (at 118.11 71.12 90)
       (effects (font (size 1.27 1.27)))
     )
@@
       (effects (font (size 1.27 1.27)))
     )
-    (property "Value" "44p" (at 100.33 87.63 90)
+    (property "Value" "47p" (at 100.33 87.63 90)
       (effects (font (size 1.27 1.27)))
     )
@@
       (effects (font (size 1.27 1.27)) (justify left))
     )
-    (property "Value" "609p" (at 107.95 97.79 0)
+    (property "Value" "620p" (at 107.95 97.79 0)
       (effects (font (size 1.27 1.27)) (justify left))
     )
@@
       (effects (font (size 1.27 1.27)) (justify left))
     )
-    (property "Value" "1218p" (at 107.95 44.45 0)
+    (property "Value" "1200p" (at 107.95 44.45 0)
       (effects (font (size 1.27 1.27)) (justify left))
     )
@@
       (effects (font (size 1.27 1.27)) (justify left))
     )
-    (property "Value" "628p" (at 92.71 44.45 0)
+    (property "Value" "620p" (at 92.71 44.45 0)
       (effects (font (size 1.27 1.27)) (justify left))
     )
@@
       (effects (font (size 1.27 1.27)))
     )
-    (property "Value" "79p" (at 118.11 123.19 90)
+    (property "Value" "82p" (at 118.11 123.19 90)
       (effects (font (size 1.27 1.27)))
     )
@@
       (effects (font (size 1.27 1.27)))
     )
-    (property "Value" "35p" (at 100.33 113.03 90)
+    (property "Value" "33p" (at 100.33 113.03 90)
       (effects (font (size 1.27 1.27)))
     )
@@
       (effects (font (size 1.27 1.27)) (justify left))
     )
-    (property "Value" "435p" (at 93.98 71.12 0)
+    (property "Value" "430p" (at 93.98 71.12 0)
       (effects (font (size 1.27 1.27)) (justify left))
     )
@@
       (effects (font (size 1.27 1.27)))
     )
-    (property "Value" "101p" (at 118.11 97.79 90)
+    (property "Value" "100p" (at 118.11 97.79 90)
       (effects (font (size 1.27 1.27)))
     )
@@
       (effects (font (size 1.27 1.27)) (justify left))
     )
-    (property "Value" "209p" (at 93.98 154.94 0)
+    (property "Value" "200p" (at 93.98 154.94 0)
       (effects (font (size 1.27 1.27)) (justify left))
     )
@@
       (effects (font (size 1.27 1.27)) (justify left))
     )
-    (property "Value" "386p" (at 130.81 71.12 0)
+    (property "Value" "390p" (at 130.81 71.12 0)
       (effects (font (size 1.27 1.27)) (justify left))
     )
@@
       (effects (font (size 1.27 1.27)) (justify left))
     )
-    (property "Value" "844p" (at 107.95 71.12 0)
+    (property "Value" "820p" (at 107.95 71.12 0)
       (effects (font (size 1.27 1.27)) (justify left))
     )
@@
       (effects (font (size 1.27 1.27)))
     )
-    (property "Value" "67p" (at 118.11 154.94 90)
+    (property "Value" "62p" (at 118.11 154.94 90)
       (effects (font (size 1.27 1.27)))
     )
@@
       (effects (font (size 1.27 1.27)))
     )
-    (property "Value" "30p" (at 100.33 144.78 90)
+    (property "Value" "33p" (at 100.33 144.78 90)
       (effects (font (size 1.27 1.27)))
     )
@@
       (effects (font (size 1.27 1.27)) (justify left))
     )
-    (property "Value" "279p" (at 130.81 97.79 0)
+    (property "Value" "270p" (at 130.81 97.79 0)
       (effects (font (size 1.27 1.27)) (justify left))
     )
@@
       (effects (font (size 1.27 1.27)) (justify left))
     )
-    (property "Value" "557p" (at 129.54 44.45 0)
+    (property "Value" "560p" (at 129.54 44.45 0)
       (effects (font (size 1.27 1.27)) (justify left))
     )
@@
       (effects (font (size 1.27 1.27)) (justify left))
     )
-    (property "Value" "474p" (at 107.95 123.19 0)
+    (property "Value" "470p" (at 107.95 123.19 0)
       (effects (font (size 1.27 1.27)) (justify left))
     )
@@
       (effects (font (size 1.27 1.27)))
     )
-    (property "Value" "89p" (at 99.06 34.29 90)
+    (property "Value" "91p" (at 99.06 34.29 90)
       (effects (font (size 1.27 1.27)))
     )
@@
       (effects (font (size 1.27 1.27)) (justify left))
     )
-    (property "Value" "217p" (at 130.81 123.19 0)
-      (effects (font (size 1.27 1.27)) (justify left))
-    )
+    (property "Value" "220p" (at 130.81 123.19 0)
+      (effects (font (size 1.27 1.27)) (justify left))
+    )
