File: 5BandCWTranceiver/qsd_revC/qsd_revC.kicad_pcb (KiCad board)
At the start: 2 copper layers, 55.9 x 37.1 mm, 56 parts, among them IC1 MCP1801, IC2 SN74LVC1G04DBVT, IC3 SN74AUP2G79DCUR, IC4 TS5A23157, IC5 SN74CBTLV3253, IC6 SN74LVC1G04DBVT, J1 Conn_Coaxial, J2 Conn_Coaxial, J3 Conn_Coaxial, Q1 J309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

Commit message: Updating field radio
Continued schematic work on field radio
Parts:
- removed C18, C21: 1nF, Capacitor_SMD:C_0603_1608Metric_Pad1.08x0.95mm_HandSolder
- removed J3: Conn_Coaxial, Connector_Coaxial:SMA_Samtec_SMA-J-P-X-ST-EM1_EdgeMount
- removed R18, R19, R26, R27: 100, Resistor_SMD:R_0603_1608Metric_Pad0.98x0.95mm_HandSolder
- removed R28: 7.5k, Resistor_SMD:R_0603_1608Metric_Pad0.98x0.95mm_HandSolder
- removed R31: 10k, Resistor_SMD:R_0603_1608Metric_Pad0.98x0.95mm_HandSolder
- removed R32: 5K, qsd_revB:RTRIM3296W
- removed U1: OPA1678, Package_SO:SOIC-8_3.9x4.9mm_P1.27mm
- added C8: 0.1uF, Capacitor_SMD:C_0603_1608Metric_Pad1.08x0.95mm_HandSolder, F.Cu at (160.9, 109.4)
- added C9: 0.1uF, Capacitor_SMD:C_0603_1608Metric_Pad1.08x0.95mm_HandSolder, F.Cu at (161.1, 115.6)
- added IC7: INA821ID, SamacSys_Parts:SOIC127P600X175-8N, F.Cu at (155.2, 117.6)
- added R11: 47k, Resistor_SMD:R_0603_1608Metric_Pad0.98x0.95mm_HandSolder, F.Cu at (143.2, 111.5)
- added R12: 47k, Resistor_SMD:R_0603_1608Metric_Pad0.98x0.95mm_HandSolder, F.Cu at (143.4, 117.5)
- added R13: 47k, Resistor_SMD:R_0603_1608Metric_Pad0.98x0.95mm_HandSolder, F.Cu at (145.4, 117.5)
- C12, C14: value 0.15uF -> 0.1uF
- C13, C15: value 0.15uF -> 470pF
- IC6: value SN74LVC1G04DBVT -> INA821ID; footprint qsd_revB:SOT95P280X145-5N -> SamacSys_Parts:SOIC127P600X175-8N
- JP9: value M03PTH -> M02PTH; footprint qsd_revB:1X03 -> qsd_revB:1X02
- R2: value 10k -> 49.9
- R3: value 5K -> 49.9; footprint qsd_revB:RTRIM3296W -> Resistor_SMD:R_0603_1608Metric_Pad0.98x0.95mm_HandSolder
- R4: value 10k -> 47k
- R8: value 4.7k -> 4.32K
- R9: value R-TRIMM3296W -> 4.32K; footprint qsd_revB:RTRIM3296W -> Resistor_SMD:R_0603_1608Metric_Pad0.98x0.95mm_HandSolder
- moved C19 37.7 mm to (126.5, 110.1), turned to 90 degrees
- moved JP8 22.7 mm to (166.8, 111.6), turned to -90 degrees
- moved IC6 20.7 mm to (155.2, 111.3)
- moved JP5 20.6 mm to (158.6, 90.7)
- moved C14 18.7 mm to (161.1, 118.3), turned to 180 degrees
- moved C12 18.1 mm to (160.9, 112.0)
- moved R9 17.3 mm to (132.3, 112.0), turned to 0 degrees
- moved R4 14.1 mm to (145.2, 111.5), turned to -90 degrees
- moved C20 9.21 mm to (166.2, 107.4)
- moved R3 7.93 mm to (149.4, 111.3), turned to -90 degrees
- moved R2 7.89 mm to (149.4, 117.5), turned to -90 degrees
- moved C15 4.79 mm to (147.4, 117.5), turned to 90 degrees
- moved C13 4.26 mm to (147.3, 111.5), turned to -90 degrees
- moved JP9 3.60 mm to (157.8, 123.0)
- moved JP3 0.89 mm to (166.8, 122.9), turned to 180 degrees
Connections:
- C12 pad 1: GND -> Net-(IC6-REF)
- C12 pad 2: /0-DEG -> GND
- C13 pad 1: GND -> /180-DEG
- C13 pad 2: /180-DEG -> /0-DEG
- C14 pad 2: /90-DEG -> Net-(IC6-REF)
- C15 pad 1: GND -> /90-DEG
- C6 pad 2: Net-(C6-Pad2) -> Net-(C7-+)
- C7 pad 1: Net-(C6-Pad2) -> Net-(C7-+)
- IC6 pad 1: unconnected-(IC6-Pad1) -> /180-DEG
- IC6 pad 2: /P1 -> Net-(IC6-RG_1)
- IC6 pad 3: GND -> Net-(IC6-RG_2)
- IC6 pad 4: Net-(IC6-Pad4) -> /0-DEG
- IC6 pad 5: /VCC3.3 -> GND
- JP8 pad 1: /I-PHASE -> Net-(IC6-OUT)
- JP8 pad 3: /Q-PHASE -> Net-(IC7-OUT)
- JP9 pad 1: /I-PHASE -> GND
- JP9 pad 2: GND -> Net-(IC6-REF)
- R2 pad 1: Net-(R2-Pad1) -> Net-(IC7-RG_1)
- R2 pad 2: /270-DEG -> Net-(IC7-RG_2)
- R3 pad 1: Net-(R3-Pad1) -> Net-(IC6-RG_1)
- R3 pad 2: Net-(C21-Pad2) -> Net-(IC6-RG_2)
- R4 pad 1: /Q-PHASE -> GND
- R4 pad 2: Net-(R3-Pad1) -> /0-DEG
- R8 pad 1: Net-(C6-Pad2) -> Net-(C7-+)
- R9 pad 1: Net-(C6-Pad2) -> GND
- R9 pad 2: GND -> Net-(C7-+)
- T1 pad 4: Net-(C6-Pad2) -> Net-(C7-+)
Routing:
- net /I-PHASE: track 43.7 -> 0.00 mm
- net Net-(C7-+): track 0.00 -> 29.3 mm
- net Net-(C6-Pad2): track 28.1 -> 0.00 mm
- net Net-(C21-Pad2): track 26.9 -> 0.00 mm, vias 1 -> 0
- net Net-(IC6-REF): track 0.00 -> 20.8 mm
- net /Q-PHASE: track 12.8 -> 0.00 mm
- net /0-DEG: track 12.8 -> 24.7 mm, vias 2 -> 4
- net Net-(C18-Pad2): track 11.7 -> 0.00 mm
- net /VCC5: track 74.6 -> 85.9 mm, vias 0 -> 1
- net /90-DEG: track 18.1 -> 28.9 mm
- net Net-(IC6-Pad4): track 10.2 -> 0.00 mm
- net Net-(IC6-OUT): track 0.00 -> 9.26 mm
- net Net-(IC7-OUT): track 0.00 -> 9.02 mm
- net Net-(R18-Pad1): track 8.90 -> 0.00 mm
- net /180-DEG: track 20.0 -> 26.9 mm, vias 4 -> 3
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Other:
- board text added: "IOUT"
- board text added: "N7WMN QSD Rev. C"
- board text added: "QOUT"
- board text added: "VBIAS"
- board text removed: "I"
- board text removed: "N7WMN Tayloe Detector Rev. C"
- board text removed: "Q"

Commit message: Tapeout PowerAmp and QSD
PowerAmp rev. C and QSD rev. D
Parts:
- moved JP6 32.5 mm to (152.5, 90.6)
- moved R10 30.2 mm to (157.3, 93.6)
- moved C7 10.2 mm to (135.4, 93.8)
- moved C6 3.38 mm to (139.1, 96.6), turned to 180 degrees
- moved IC2 2.58 mm to (148.5, 97.3), turned to 0 degrees
Routing:
- net /VCC5: track 85.9 -> 108.1 mm
- net /SIDEBAND: track 41.7 -> 27.0 mm, vias 4 -> 3
- net Net-(C7-+): track 29.3 -> 24.1 mm
- net Net-(IC2-Y): track 5.49 -> 2.24 mm
- net /P1: track 22.5 -> 21.7 mm
- net /VCC3.3: track 37.7 -> 38.2 mm
- net /180-DEG: track 26.9 -> 26.6 mm, vias 3 -> 2
- net GND: vias 46 -> 52
Other:
- board text added: "N7WMN QSD Rev. D"
- board text removed: "N7WMN QSD Rev. C"
