File: fieldRadio/powerInput.kicad_sch (KiCad schematic)
At the start: 7 parts, among them Q1 IRF9540, U1 LM1085-5.0

Commit message: More schematic dev.
More schematic development
Parts:
- renumbered C1 to C146, C2 to C147, C3 to C148, C4 to C149, Q1 to Q25, U1 to U11
Changed lines of the file:
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@@
   (symbol (lib_id "Device:C_Polarized_US") (at 245.11 146.05 0) (unit 1)
     (in_bom yes) (on_board yes) (dnp no)
-    (property "Reference" "C3" (at 245.11 143.51 0)
+    (property "Reference" "C148" (at 245.11 143.51 0)
       (effects (font (size 1.27 1.27)) (justify left))
     )
@@
       (project "fieldRadio"
         (path "/a1d1b2b0-2f27-4dc0-94ba-bb0e02933617/56bfcbb6-5b4c-41a3-a0f1-0c3e063460f4"
+          (reference "C148") (unit 1)
+        )
+      )
+      (project ""
+        (path "/fdb52485-f59b-413f-ad63-5c01cdc03d56"
           (reference "C3") (unit 1)
         )
       )
-      (project ""
-        (path "/fdb52485-f59b-413f-ad63-5c01cdc03d56"
-          (reference "C3") (unit 1)
-        )
-      )
     )
   )
   (symbol (lib_id "Device:C") (at 219.71 146.05 0) (unit 1)
     (in_bom yes) (on_board yes) (dnp no)
-    (property "Reference" "C2" (at 220.98 143.51 0)
+    (property "Reference" "C147" (at 220.98 143.51 0)
       (effects (font (size 1.27 1.27)) (justify left))
     )
@@
       (project "fieldRadio"
         (path "/a1d1b2b0-2f27-4dc0-94ba-bb0e02933617/56bfcbb6-5b4c-41a3-a0f1-0c3e063460f4"
+          (reference "C147") (unit 1)
+        )
+      )
+      (project ""
+        (path "/fdb52485-f59b-413f-ad63-5c01cdc03d56"
           (reference "C2") (unit 1)
         )
       )
-      (project ""
-        (path "/fdb52485-f59b-413f-ad63-5c01cdc03d56"
-          (reference "C2") (unit 1)
-        )
-      )
     )
   )
   (symbol (lib_id "Regulator_Linear:LM1085-5.0") (at 232.41 139.7 0) (unit 1)
     (in_bom yes) (on_board yes) (dnp no) (fields_autoplaced)
-    (property "Reference" "U1" (at 232.41 132.08 0)
+    (property "Reference" "U11" (at 232.41 132.08 0)
       (effects (font (size 1.27 1.27)))
     )
@@
       (project "fieldRadio"
         (path "/a1d1b2b0-2f27-4dc0-94ba-bb0e02933617/56bfcbb6-5b4c-41a3-a0f1-0c3e063460f4"
+          (reference "U11") (unit 1)
+        )
+      )
+      (project ""
+        (path "/fdb52485-f59b-413f-ad63-5c01cdc03d56"
           (reference "U1") (unit 1)
         )
       )
-      (project ""
-        (path "/fdb52485-f59b-413f-ad63-5c01cdc03d56"
-          (reference "U1") (unit 1)
-        )
-      )
     )
   )
   (symbol (lib_id "Device:Q_PMOS_GDS") (at 173.355 128.905 90) (unit 1)
     (in_bom yes) (on_board yes) (dnp no) (fields_autoplaced)
-    (property "Reference" "Q1" (at 173.355 118.745 90)
+    (property "Reference" "Q25" (at 173.355 118.745 90)
       (effects (font (size 1.27 1.27)))
     )
@@
       (project "fieldRadio"
         (path "/a1d1b2b0-2f27-4dc0-94ba-bb0e02933617/56bfcbb6-5b4c-41a3-a0f1-0c3e063460f4"
+          (reference "Q25") (unit 1)
+        )
+      )
+      (project ""
+        (path "/fdb52485-f59b-413f-ad63-5c01cdc03d56"
           (reference "Q1") (unit 1)
         )
       )
-      (project ""
-        (path "/fdb52485-f59b-413f-ad63-5c01cdc03d56"
-          (reference "Q1") (unit 1)
-        )
-      )
     )
   )
   (symbol (lib_id "Device:C") (at 255.27 146.05 0) (unit 1)
     (in_bom yes) (on_board yes) (dnp no)
-    (property "Reference" "C4" (at 256.54 143.51 0)
+    (property "Reference" "C149" (at 256.54 143.51 0)
       (effects (font (size 1.27 1.27)) (justify left))
     )
@@
       (project "fieldRadio"
         (path "/a1d1b2b0-2f27-4dc0-94ba-bb0e02933617/56bfcbb6-5b4c-41a3-a0f1-0c3e063460f4"
+          (reference "C149") (unit 1)
+        )
+      )
+      (project ""
+        (path "/fdb52485-f59b-413f-ad63-5c01cdc03d56"
           (reference "C4") (unit 1)
         )
       )
-      (project ""
-        (path "/fdb52485-f59b-413f-ad63-5c01cdc03d56"
-          (reference "C4") (unit 1)
-        )
-      )
     )
   )
@@
   (symbol (lib_id "Device:C_Polarized_US") (at 208.28 146.05 0) (unit 1)
     (in_bom yes) (on_board yes) (dnp no)
-    (property "Reference" "C1" (at 209.55 143.51 0)
+    (property "Reference" "C146" (at 209.55 143.51 0)
       (effects (font (size 1.27 1.27)) (justify left))
     )
@@
       (project "fieldRadio"
         (path "/a1d1b2b0-2f27-4dc0-94ba-bb0e02933617/56bfcbb6-5b4c-41a3-a0f1-0c3e063460f4"
+          (reference "C146") (unit 1)
+        )
+      )
+      (project ""
+        (path "/fdb52485-f59b-413f-ad63-5c01cdc03d56"
           (reference "C1") (unit 1)
         )
       )
-      (project ""
-        (path "/fdb52485-f59b-413f-ad63-5c01cdc03d56"
-          (reference "C1") (unit 1)
-        )
-      )
     )
   )
   (symbol (lib_id "power:GND") (at 208.28 156.21 0) (unit 1)
     (in_bom yes) (on_board yes) (dnp no) (fields_autoplaced)
-    (property "Reference" "#PWR01" (at 208.28 162.56 0)
+    (property "Reference" "#PWR032" (at 208.28 162.56 0)
       (effects (font (size 1.27 1.27)) hide)
     )
@@
       (project "fieldRadio"
         (path "/a1d1b2b0-2f27-4dc0-94ba-bb0e02933617/56bfcbb6-5b4c-41a3-a0f1-0c3e063460f4"
-          (reference "#PWR01") (unit 1)
-        )
-      )
+          (reference "#PWR032") (unit 1)
+        )
+      )

Commit message: Update Connectors
Changed to PCB mount connectors for back panel
Changed lines of the file:
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@@
     (effects (font (size 1.27 1.27)) (justify left bottom))
   )
-  (global_label "VDD12" (shape bidirectional) (at 201.295 139.7 180) (fields_autoplaced)
+  (global_label "VDD12" (shape input) (at 201.295 139.7 180) (fields_autoplaced)
     (effects (font (size 1.27 1.27)) (justify right))
-    (property "Intersheetrefs" "${INTERSHEET_REFS}" (at 191.6924 139.7 0)
+    (property "Intersheetrefs" "${INTERSHEET_REFS}" (at 192.8037 139.7 0)
       (effects (font (size 1.27 1.27)) (justify right))
     )
   )
-  (hierarchical_label "PWR_IN" (shape bidirectional) (at 161.925 126.365 180) (fields_autoplaced)
+  (hierarchical_label "PWR_IN" (shape input) (at 161.925 126.365 180) (fields_autoplaced)
     (effects (font (size 1.27 1.27)) (justify right))
   )
-  (hierarchical_label "+5V" (shape bidirectional) (at 269.24 139.7 0) (fields_autoplaced)
+  (hierarchical_label "+5V" (shape output) (at 269.24 139.7 0) (fields_autoplaced)
     (effects (font (size 1.27 1.27)) (justify left))
   )

Commit message: Clean Up
Schematic clean up in prep for layout
Parts:
- renumbered C146 to C153, C147 to C154, C148 to C155, C149 to C156, Q25 to Q21, U11 to U10
Changed lines of the file:
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@@
     (effects (font (size 1.27 1.27)) (justify left))
   )
-  (hierarchical_label "PWR_SWTCH" (shape bidirectional) (at 211.455 126.365 0) (fields_autoplaced)
+  (hierarchical_label "PWR_SWTCH" (shape output) (at 211.455 126.365 0) (fields_autoplaced)
     (effects (font (size 1.27 1.27)) (justify left))
   )
   (symbol (lib_id "Device:C_Polarized_US") (at 245.11 146.05 0) (unit 1)
     (in_bom yes) (on_board yes) (dnp no)
-    (property "Reference" "C148" (at 245.11 143.51 0)
+    (property "Reference" "C155" (at 245.11 143.51 0)
       (effects (font (size 1.27 1.27)) (justify left))
     )
@@
       (project "fieldRadio"
         (path "/a1d1b2b0-2f27-4dc0-94ba-bb0e02933617/56bfcbb6-5b4c-41a3-a0f1-0c3e063460f4"
-          (reference "C148") (unit 1)
+          (reference "C155") (unit 1)
         )
       )
@@
   (symbol (lib_id "Device:C") (at 219.71 146.05 0) (unit 1)
     (in_bom yes) (on_board yes) (dnp no)
-    (property "Reference" "C147" (at 220.98 143.51 0)
+    (property "Reference" "C154" (at 220.98 143.51 0)
       (effects (font (size 1.27 1.27)) (justify left))
     )
@@
       (project "fieldRadio"
         (path "/a1d1b2b0-2f27-4dc0-94ba-bb0e02933617/56bfcbb6-5b4c-41a3-a0f1-0c3e063460f4"
-          (reference "C147") (unit 1)
+          (reference "C154") (unit 1)
         )
       )
@@
   (symbol (lib_id "Regulator_Linear:LM1085-5.0") (at 232.41 139.7 0) (unit 1)
     (in_bom yes) (on_board yes) (dnp no) (fields_autoplaced)
-    (property "Reference" "U11" (at 232.41 132.08 0)
+    (property "Reference" "U10" (at 232.41 132.08 0)
       (effects (font (size 1.27 1.27)))
     )
@@
       (project "fieldRadio"
         (path "/a1d1b2b0-2f27-4dc0-94ba-bb0e02933617/56bfcbb6-5b4c-41a3-a0f1-0c3e063460f4"
-          (reference "U11") (unit 1)
+          (reference "U10") (unit 1)
         )
       )
@@
   (symbol (lib_id "Device:Q_PMOS_GDS") (at 173.355 128.905 90) (unit 1)
     (in_bom yes) (on_board yes) (dnp no) (fields_autoplaced)
-    (property "Reference" "Q25" (at 173.355 118.745 90)
+    (property "Reference" "Q21" (at 173.355 118.745 90)
       (effects (font (size 1.27 1.27)))
     )
@@
       (project "fieldRadio"
         (path "/a1d1b2b0-2f27-4dc0-94ba-bb0e02933617/56bfcbb6-5b4c-41a3-a0f1-0c3e063460f4"
-          (reference "Q25") (unit 1)
+          (reference "Q21") (unit 1)
         )
       )
@@
   (symbol (lib_id "Device:C") (at 255.27 146.05 0) (unit 1)
     (in_bom yes) (on_board yes) (dnp no)
-    (property "Reference" "C149" (at 256.54 143.51 0)
+    (property "Reference" "C156" (at 256.54 143.51 0)
       (effects (font (size 1.27 1.27)) (justify left))
     )
@@
       (project "fieldRadio"
         (path "/a1d1b2b0-2f27-4dc0-94ba-bb0e02933617/56bfcbb6-5b4c-41a3-a0f1-0c3e063460f4"
-          (reference "C149") (unit 1)
+          (reference "C156") (unit 1)
         )
       )
@@
   (symbol (lib_id "Device:C_Polarized_US") (at 208.28 146.05 0) (unit 1)
     (in_bom yes) (on_board yes) (dnp no)
-    (property "Reference" "C146" (at 209.55 143.51 0)
+    (property "Reference" "C153" (at 209.55 143.51 0)
       (effects (font (size 1.27 1.27)) (justify left))
     )
@@
       (project "fieldRadio"
         (path "/a1d1b2b0-2f27-4dc0-94ba-bb0e02933617/56bfcbb6-5b4c-41a3-a0f1-0c3e063460f4"
-          (reference "C146") (unit 1)
+          (reference "C153") (unit 1)
         )
       )
@@
   (symbol (lib_id "power:GND") (at 208.28 156.21 0) (unit 1)
     (in_bom yes) (on_board yes) (dnp no) (fields_autoplaced)
-    (property "Reference" "#PWR032" (at 208.28 162.56 0)
+    (property "Reference" "#PWR039" (at 208.28 162.56 0)
       (effects (font (size 1.27 1.27)) hide)
     )
@@
       (project "fieldRadio"
         (path "/a1d1b2b0-2f27-4dc0-94ba-bb0e02933617/56bfcbb6-5b4c-41a3-a0f1-0c3e063460f4"
-          (reference "#PWR032") (unit 1)
-        )
-      )
+          (reference "#PWR039") (unit 1)
+        )
+      )
