File: fieldRadio/hplp_filters.kicad_sch (KiCad schematic)
At the start: 0 parts

Commit message: Updating field radio
Continued schematic work on field radio
Parts:
- added C15: 0.82uF, Capacitor_SMD:C_0603_1608Metric_Pad1.08x0.95mm_HandSolder, symbol Device:C
- added C16: 0.39uF, Capacitor_SMD:C_0603_1608Metric_Pad1.08x0.95mm_HandSolder, symbol Device:C
- added C17, C26, C32, C35, C38: 0.012uF, Capacitor_SMD:C_0603_1608Metric_Pad1.08x0.95mm_HandSolder, symbol Device:C
- added C18, C27, C33, C39: 0.0033uF, Capacitor_SMD:C_0603_1608Metric_Pad1.08x0.95mm_HandSolder, symbol Device:C
- added C19: 0.015uF, Capacitor_SMD:C_0603_1608Metric_Pad1.08x0.95mm_HandSolder, symbol Device:C
- added C20: 0.0039uF, Capacitor_SMD:C_0603_1608Metric_Pad1.08x0.95mm_HandSolder, symbol Device:C
- added C21, C22, C24, C41: 0.1uF, Capacitor_SMD:C_0603_1608Metric_Pad1.08x0.95mm_HandSolder, symbol Device:C
- added C23: 1uF, Capacitor_SMD:C_0603_1608Metric_Pad1.08x0.95mm_HandSolder, symbol Device:C
- added C25, C36: 0.47uF, Capacitor_SMD:C_0603_1608Metric_Pad1.08x0.95mm_HandSolder, symbol Device:C
- added C28: 0.018uF, Capacitor_SMD:C_0603_1608Metric_Pad1.08x0.95mm_HandSolder, symbol Device:C
- added C29: 0.0056uF, Capacitor_SMD:C_0603_1608Metric_Pad1.08x0.95mm_HandSolder, symbol Device:C
- added C30: 1.5uF, Capacitor_SMD:C_0603_1608Metric_Pad1.08x0.95mm_HandSolder, symbol Device:C
- added C31: 0.68uF, Capacitor_SMD:C_0603_1608Metric_Pad1.08x0.95mm_HandSolder, symbol Device:C
- added C34: 0.039uF, Capacitor_SMD:C_0603_1608Metric_Pad1.08x0.95mm_HandSolder, symbol Device:C
- added C37: 0.22uF, Capacitor_SMD:C_0603_1608Metric_Pad1.08x0.95mm_HandSolder, symbol Device:C
- added C40: 0.33uF, Capacitor_SMD:C_0603_1608Metric_Pad1.08x0.95mm_HandSolder, symbol Device:C
- added R24: 9.53K, Resistor_SMD:R_0603_1608Metric_Pad0.98x0.95mm_HandSolder, symbol Device:R_US
- added R25: 10.5K, Resistor_SMD:R_0603_1608Metric_Pad0.98x0.95mm_HandSolder, symbol Device:R_US
- added R26: 23.2K, Resistor_SMD:R_0603_1608Metric_Pad0.98x0.95mm_HandSolder, symbol Device:R_US
- added R27: 21K, Resistor_SMD:R_0603_1608Metric_Pad0.98x0.95mm_HandSolder, symbol Device:R_US
- added R28, R40: 1.02K, Resistor_SMD:R_0603_1608Metric_Pad0.98x0.95mm_HandSolder, symbol Device:R_US
- added R29: 866, Resistor_SMD:R_0603_1608Metric_Pad0.98x0.95mm_HandSolder, symbol Device:R_US
- added R30: 11K, Resistor_SMD:R_0603_1608Metric_Pad0.98x0.95mm_HandSolder, symbol Device:R_US
- added R31: 8.06K, Resistor_SMD:R_0603_1608Metric_Pad0.98x0.95mm_HandSolder, symbol Device:R_US
- added R32: 16.5K, Resistor_SMD:R_0603_1608Metric_Pad0.98x0.95mm_HandSolder, symbol Device:R_US
- added R33: 18.7K, Resistor_SMD:R_0603_1608Metric_Pad0.98x0.95mm_HandSolder, symbol Device:R_US
- added R34: 1K, Resistor_SMD:R_0603_1608Metric_Pad0.98x0.95mm_HandSolder, symbol Device:R_US
- added R35: 604, Resistor_SMD:R_0603_1608Metric_Pad0.98x0.95mm_HandSolder, symbol Device:R_US
- added R36: 8.66K, Resistor_SMD:R_0603_1608Metric_Pad0.98x0.95mm_HandSolder, symbol Device:R_US
- added R37: 6.04K, Resistor_SMD:R_0603_1608Metric_Pad0.98x0.95mm_HandSolder, symbol Device:R_US
- added R38: 9.76K, Resistor_SMD:R_0603_1608Metric_Pad0.98x0.95mm_HandSolder, symbol Device:R_US
- added R39: 11.8K, Resistor_SMD:R_0603_1608Metric_Pad0.98x0.95mm_HandSolder, symbol Device:R_US
- added R41: 267, Resistor_SMD:R_0603_1608Metric_Pad0.98x0.95mm_HandSolder, symbol Device:R_US
- added R42: 2.55K, Resistor_SMD:R_0603_1608Metric_Pad0.98x0.95mm_HandSolder, symbol Device:R_US
- added R43: 1.96K, Resistor_SMD:R_0603_1608Metric_Pad0.98x0.95mm_HandSolder, symbol Device:R_US
- added R44: 3.92K, Resistor_SMD:R_0603_1608Metric_Pad0.98x0.95mm_HandSolder, symbol Device:R_US
- added R45: 4.32K, Resistor_SMD:R_0603_1608Metric_Pad0.98x0.95mm_HandSolder, symbol Device:R_US
- added R46: 9.09K, Resistor_SMD:R_0603_1608Metric_Pad0.98x0.95mm_HandSolder, symbol Device:R_US
- added R47: 301, Resistor_SMD:R_0603_1608Metric_Pad0.98x0.95mm_HandSolder, symbol Device:R_US
- added U5, U7: OPA1679, Package_SO:SOIC-14_3.9x8.7mm_P1.27mm, symbol Amplifier_Operational:OPA1679
- added U6: OPA1679, symbol Amplifier_Operational:OPA1679
Connections:
- new net: C38.1, R44.2, U6.5 (+)
- new net: C41.1, R43.2, R45.1
- new net: C39.1, R45.2, U7.5 (+)
- new net: C20.2, R31.1, U7.1, U7.2 (-)
- new net: C29.1, R31.2, R33.1
- new net: C31.2, R40.2, U5.10 (+)
- new net: C36.1, R41.2, U5.8, U5.9 (-)
- new net: C28.2, R36.1, U6.13 (-), U6.14
- new net: C34.1, R36.2, R38.1
- new net: C27.1, R33.2, U7.12 (+)
- new net: C29.2, R37.1, U7.13 (-), U7.14
- new net: C25.2, R34.2, U5.12 (+)
- new net: R24.1, R25.1, R47.2, U5.6 (-), U5.7
- new net: C20.1, R25.2, R27.1
- new net: C34.2, R42.1, U6.8, U6.9 (-)
- new net: C32.1, R38.2, U6.10 (+)
- new net: C23.2, C25.1, R35.1
- new net: C30.1, R35.2, U5.13 (-), U5.14
- new net: C40.1, R42.2, R44.1
- new net: C23.1, R29.2, U5.1, U5.2 (-)
- new net: C35.1, R37.2, R39.1
- new net: C35.2, R43.1, U7.8, U7.9 (-)
- new net: C19.1, R24.2, R26.1
- new net: C17.1, R26.2, U6.3 (+)
- new net: C16.2, R28.2, U5.3 (+)
- new net: C30.2, C31.1, R41.1
- new net: C36.2, C37.1, R47.1
- new net: C18.1, R27.2, U7.3 (+)
- new net: C33.1, R39.2, U7.10 (+)
- new net: C15.2, C16.1, R29.1
- new net: C37.2, R46.2, U5.5 (+)
- new net: C28.1, R30.2, R32.1
- new net: C26.1, R32.2, U6.12 (+)
- new net: C19.2, R30.1, U6.1, U6.2 (-)
- new net GND: C17.2, C18.2, C21.1, C22.1, C24.1, C26.2, C27.2, C32.2, C33.2, C38.2, C39.2, U5.11 (V-), U6.11 (V-), U7.11 (V-)
- new net VDD5: C21.2, C22.2, C24.2, U5.4 (V+), U6.4 (V+), U7.4 (V+)
- new net in: C15.1
- new net narrow: C40.2, U6.6 (-), U6.7
- new net vbias: R28.1, R34.1, R40.1, R46.1
- new net wide: C41.2, U7.6 (-), U7.7
Other:
- note added: "300 Hz High Pass"
- note added: "3kHz Low Pass"
- note added: "800 Hz Low Pass"
- note added: "All Pass Filter and Wide/Narrow Audio Filters"

Commit message: More schematic dev.
More schematic development
Parts:
- renumbered C15 to C150, C16 to C151, C17 to C152, C18 to C153, C19 to C154, C20 to C155, C21 to C156, C22 to C157, C23 to C158, C24 to C159, C25 to C160, C26 to C161, C27 to C162, C28 to C163, C29 to C164, C30 to C165, C31 to C166, C32 to C167, C33 to C168, C34 to C169, C35 to C170, C36 to C171, C37 to C172, C38 to C173, C39 to C174, C40 to C175, C41 to C176, R24 to R156, R25 to R157, R26 to R158, R27 to R159, R28 to R160, R29 to R161, R30 to R162, R31 to R163, R32 to R164, R33 to R165, R34 to R166, R35 to R167, R36 to R168, R37 to R169, R38 to R170, R39 to R171, R40 to R172, R41 to R173, R42 to R174, R43 to R175, R44 to R176, R45 to R177, R46 to R178, R47 to R179, U5 to U12, U6 to U13, U7 to U14

Commit message: Clean Up
Schematic clean up in prep for layout
Parts:
- renumbered C150 to C157, C151 to C158, C152 to C159, C153 to C160, C154 to C161, C155 to C162, C156 to C163, C157 to C164, C158 to C165, C159 to C166, C160 to C167, C161 to C168, C162 to C169, C163 to C170, C164 to C171, C165 to C172, C166 to C173, C167 to C174, C168 to C175, C169 to C176, C170 to C177, C171 to C178, C172 to C179, C173 to C180, C174 to C181, C175 to C182, C176 to C183, R156 to R149, R157 to R150, R158 to R151, R159 to R152, R160 to R153, R161 to R154, R162 to R155, R163 to R156, R164 to R157, R165 to R158, R166 to R159, R167 to R160, R168 to R161, R169 to R162, R170 to R163, R171 to R164, R172 to R165, R173 to R166, R174 to R167, R175 to R168, R176 to R169, R177 to R170, R178 to R171, R179 to R172, U12 to U11, U13 to U12, U14 to U13

Commit message: Placement Update
LPF and TR Switch placed
Parts:
- U11, U12, U13: footprint (none) -> Package_SO:SOIC-14_3.9x8.7mm_P1.27mm
Changed lines of the file:
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@@
       (effects (font (size 1.27 1.27)) (justify left))
     )
-    (property "Footprint" "" (at 45.72 176.53 0)
+    (property "Footprint" "Package_SO:SOIC-14_3.9x8.7mm_P1.27mm" (at 45.72 176.53 0)
       (effects (font (size 1.27 1.27)) hide)
     )
@@
       (effects (font (size 1.27 1.27)) (justify left))
     )
-    (property "Footprint" "" (at 31.75 175.26 0)
+    (property "Footprint" "Package_SO:SOIC-14_3.9x8.7mm_P1.27mm" (at 31.75 175.26 0)
       (effects (font (size 1.27 1.27)) hide)
     )
@@
       (effects (font (size 1.27 1.27)) (justify left))
     )
-    (property "Footprint" "" (at 59.69 176.53 0)
-      (effects (font (size 1.27 1.27)) hide)
-    )
+    (property "Footprint" "Package_SO:SOIC-14_3.9x8.7mm_P1.27mm" (at 59.69 176.53 0)
+      (effects (font (size 1.27 1.27)) hide)
+    )
