File: fieldRadio/powerAmp.kicad_sch (KiCad schematic)
At the start: 41 parts, among them IC1 UCC27517DBVR, IC2 UCC27517DBVR, Q1 NSS1C301ET4G, Q2 DMN10H220LPDW, T1 1:1, U3 MIC5235-5.0YM5

Commit message: Finished Groups
Blocks are placed
Parts:
- R10: now not fitted
Connections:
- net GND: now also C15.2, C17.2, C19.1, IC1.2 (GND), IC1.4 (IN-), IC2.2 (GND), R15.2, U$2.11 (V-)
Changed lines of the file:
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@@
-    )
-  )
-  (symbol (lib_id "powerAmp_RevB-eagle-import:GND") (at 297.18 59.055 0) (unit 1)
-    (in_bom yes) (on_board yes) (dnp no)
-    (property "Reference" "#SUPPLY02" (at 297.18 59.055 0)
-      (effects (font (size 1.27 1.27)) hide)
-    )
-    (property "Value" "GND" (at 295.275 62.23 0)
-      (effects (font (size 1.778 1.5113)) (justify left bottom))
-    )
-    (property "Footprint" "powerAmp_RevB:" (at 297.18 59.055 0)
-      (effects (font (size 1.27 1.27)) hide)
-    )
-    (property "Datasheet" "" (at 297.18 59.055 0)
-      (effects (font (size 1.27 1.27)) hide)
-    )
-    (pin "1")
-    (instances
-      (project "fieldRadio"
-        (path "/a1d1b2b0-2f27-4dc0-94ba-bb0e02933617/de17e96d-acc8-4488-9767-c0e10e15a863"
-          (reference "#SUPPLY09") (unit 1)
-        )
-      )
-      (project ""
-        (path "/c58960d9-4cac-4036-ad2e-1aef26946dae"
-          (reference "#SUPPLY02") (unit 1)
-        )
-      )
-      (project "powerAmp"
-        (path "/c63d077a-bb30-4740-8b96-a434a85a3a02"
-          (reference "#SUPPLY02") (unit 1)
-        )
-      )
     )
   )
@@
     )
   )
-  (symbol (lib_name "GND_2") (lib_id "powerAmp_RevB-eagle-import:GND") (at 149.225 185.42 0) (unit 1)
-    (in_bom yes) (on_board yes) (dnp no)
-    (property "Reference" "#SUPPLY011" (at 149.225 185.42 0)
-      (effects (font (size 1.27 1.27)) hide)
-    )
-    (property "Value" "GND" (at 147.32 188.595 0)
-      (effects (font (size 1.778 1.5113)) (justify left bottom))
-    )
-    (property "Footprint" "powerAmp_RevB:" (at 149.225 185.42 0)
-      (effects (font (size 1.27 1.27)) hide)
-    )
-    (property "Datasheet" "" (at 149.225 185.42 0)
-      (effects (font (size 1.27 1.27)) hide)
-    )
-    (pin "1")
-    (instances
-      (project "fieldRadio"
-        (path "/a1d1b2b0-2f27-4dc0-94ba-bb0e02933617/de17e96d-acc8-4488-9767-c0e10e15a863"
-          (reference "#SUPPLY05") (unit 1)
-        )
-      )
-      (project "powerAmp"
-        (path "/c63d077a-bb30-4740-8b96-a434a85a3a02"
-          (reference "#SUPPLY011") (unit 1)
+  (symbol (lib_id "powerAmp_RevB-eagle-import:GND") (at 149.86 102.235 0) (unit 1)
+    (in_bom yes) (on_board yes) (dnp no)
+    (property "Reference" "#SUPPLY06" (at 149.86 102.235 0)
+      (effects (font (size 1.27 1.27)) hide)
+    )
+    (property "Value" "GND" (at 147.955 105.41 0)
+      (effects (font (size 1.778 1.5113)) (justify left bottom))
+    )
+    (property "Footprint" "powerAmp_RevB:" (at 149.86 102.235 0)
+      (effects (font (size 1.27 1.27)) hide)
+    )
+    (property "Datasheet" "" (at 149.86 102.235 0)
+      (effects (font (size 1.27 1.27)) hide)
+    )
+    (pin "1")
+    (instances
+      (project "fieldRadio"
+        (path "/a1d1b2b0-2f27-4dc0-94ba-bb0e02933617/de17e96d-acc8-4488-9767-c0e10e15a863"
+          (reference "#SUPPLY06") (unit 1)
         )
       )
@@
         (path "/c63d077a-bb30-4740-8b96-a434a85a3a02"
           (reference "U$2") (unit 5)
+        )
+      )
+    )
+  )
+  (symbol (lib_id "powerAmp_RevB-eagle-import:GND") (at 297.18 59.055 0) (unit 1)
+    (in_bom yes) (on_board yes) (dnp no)
+    (property "Reference" "#SUPPLY09" (at 297.18 59.055 0)
+      (effects (font (size 1.27 1.27)) hide)
+    )
+    (property "Value" "GND" (at 295.275 62.23 0)
+      (effects (font (size 1.778 1.5113)) (justify left bottom))
+    )
+    (property "Footprint" "powerAmp_RevB:" (at 297.18 59.055 0)
+      (effects (font (size 1.27 1.27)) hide)
+    )
+    (property "Datasheet" "" (at 297.18 59.055 0)
+      (effects (font (size 1.27 1.27)) hide)
+    )
+    (pin "1")
+    (instances
+      (project "fieldRadio"
+        (path "/a1d1b2b0-2f27-4dc0-94ba-bb0e02933617/de17e96d-acc8-4488-9767-c0e10e15a863"
+          (reference "#SUPPLY09") (unit 1)
         )
       )
@@
     )
   )
-  (symbol (lib_name "GND_1") (lib_id "powerAmp_RevB-eagle-import:GND") (at 149.86 102.235 0) (unit 1)
-    (in_bom yes) (on_board yes) (dnp no)
-    (property "Reference" "#SUPPLY08" (at 149.86 102.235 0)
-      (effects (font (size 1.27 1.27)) hide)
-    )
-    (property "Value" "GND" (at 147.955 105.41 0)
-      (effects (font (size 1.778 1.5113)) (justify left bottom))
-    )
-    (property "Footprint" "powerAmp_RevB:" (at 149.86 102.235 0)
-      (effects (font (size 1.27 1.27)) hide)
-    )
-    (property "Datasheet" "" (at 149.86 102.235 0)
-      (effects (font (size 1.27 1.27)) hide)
-    )
-    (pin "1")
-    (instances
-      (project "fieldRadio"
-        (path "/a1d1b2b0-2f27-4dc0-94ba-bb0e02933617/de17e96d-acc8-4488-9767-c0e10e15a863"
-          (reference "#SUPPLY06") (unit 1)
-        )
-      )
-      (project ""
-        (path "/c58960d9-4cac-4036-ad2e-1aef26946dae"
-          (reference "#SUPPLY08") (unit 1)
-        )
-      )
-      (project "powerAmp"
-        (path "/c63d077a-bb30-4740-8b96-a434a85a3a02"
-          (reference "#SUPPLY08") (unit 1)
-        )
-      )
-    )
-  )
   (symbol (lib_id "powerAmp_RevB-eagle-import:CAP_POLPTH1") (at 274.32 46.355 0) (unit 1)
     (in_bom yes) (on_board yes) (dnp no)
@@
       (effects (font (size 1.778 1.5113)) (justify left bottom))
     )
-    (property "Value" "CAP_POLPTH1" (at 275.336 50.546 0)
+    (property "Value" "CAP_POLPTH1" (at 258.445 51.435 0)
       (effects (font (size 1.778 1.5113)) (justify left bottom))
     )
@@
         (path "/c63d077a-bb30-4740-8b96-a434a85a3a02"
           (reference "C4") (unit 1)
+        )
+      )
+    )
+  )
+  (symbol (lib_id "powerAmp_RevB-eagle-import:GND") (at 149.225 185.42 0) (unit 1)
+    (in_bom yes) (on_board yes) (dnp no)
+    (property "Reference" "#SUPPLY05" (at 149.225 185.42 0)
+      (effects (font (size 1.27 1.27)) hide)
+    )
+    (property "Value" "GND" (at 147.32 188.595 0)
+      (effects (font (size 1.778 1.5113)) (justify left bottom))
+    )
+    (property "Footprint" "powerAmp_RevB:" (at 149.225 185.42 0)
+      (effects (font (size 1.27 1.27)) hide)
+    )
+    (property "Datasheet" "" (at 149.225 185.42 0)
+      (effects (font (size 1.27 1.27)) hide)
+    )
+    (pin "1")
+    (instances
+      (project "fieldRadio"
+        (path "/a1d1b2b0-2f27-4dc0-94ba-bb0e02933617/de17e96d-acc8-4488-9767-c0e10e15a863"
+          (reference "#SUPPLY05") (unit 1)
         )
       )
@@
   )
   (symbol (lib_id "powerAmp_RevB-eagle-import:RESISTOR0603-RES") (at 290.195 83.185 180) (unit 1)
-    (in_bom yes) (on_board yes) (dnp no)
+    (in_bom yes) (on_board yes) (dnp yes)
     (property "Reference" "R10" (at 282.575 82.4484 0)
       (effects (font (size 1.778 1.5113)) (justify right top))
@@
       (effects (font (size 1.27 1.27)) hide)
     )
+    (property "Mouser Part Number" "" (at 290.195 83.185 0)
+      (effects (font (size 1.27 1.27)) hide)
+    )

Commit message: Placement Refinement 1
Ungrouping blocks and optimizing placement
Parts:
- removed C9: CAP_POLPTH1, Capacitor_THT:C_Radial_D5.0mm_H11.0mm_P2.00mm, symbol powerAmp_RevB-eagle-import:CAP_POLPTH1
- L1: footprint Transformer_THT:Autotransformer_Toroid_1Tap_Horizontal_D14.0mm_Amidon-T50 -> Transformer_THT:Transformer_Toroid_Horizontal_D14.0mm_Amidon-T50
Changed lines of the file:
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@@
   (junction (at 297.18 38.735) (diameter 0) (color 0 0 0 0)
   )
-  (junction (at 284.48 38.735) (diameter 0) (color 0 0 0 0)
-  )
   (junction (at 170.18 97.155) (diameter 0) (color 0 0 0 0)
   )
@@
   )
   (junction (at 149.225 178.435) (diameter 0) (color 0 0 0 0)
-  )
-  (junction (at 284.48 53.975) (diameter 0) (color 0 0 0 0)
   )
   (junction (at 103.505 128.27) (diameter 0) (color 0 0 0 0)
@@
     (stroke (width 0) (type default))
   )
-  (wire (pts (xy 274.32 43.815) (xy 274.32 38.735))
-    (stroke (width 0) (type default))
-  )
   (wire (pts (xy 264.16 177.165) (xy 264.16 170.815))
     (stroke (width 0) (type default))
@@
     (stroke (width 0) (type default))
   )
-  (wire (pts (xy 274.32 51.435) (xy 274.32 53.975))
-    (stroke (width 0) (type default))
-  )
   (wire (pts (xy 307.34 103.505) (xy 313.69 103.505))
     (stroke (width 0) (type default))
@@
     (stroke (width 0) (type default))
   )
-  (wire (pts (xy 274.32 38.735) (xy 284.48 38.735))
-    (stroke (width 0) (type default))
-  )
   (wire (pts (xy 269.875 83.185) (xy 269.875 85.725))
     (stroke (width 0) (type default))
@@
   )
   (wire (pts (xy 264.16 170.815) (xy 259.08 170.815))
-    (stroke (width 0) (type default))
-  )
-  (wire (pts (xy 274.32 53.975) (xy 284.48 53.975))
     (stroke (width 0) (type default))
   )
@@
     )
   )
-  (symbol (lib_id "powerAmp_RevB-eagle-import:CAP_POLPTH1") (at 274.32 46.355 0) (unit 1)
-    (in_bom yes) (on_board yes) (dnp no)
-    (property "Reference" "C9" (at 275.336 45.72 0)
-      (effects (font (size 1.778 1.5113)) (justify left bottom))
-    )
-    (property "Value" "CAP_POLPTH1" (at 258.445 51.435 0)
-      (effects (font (size 1.778 1.5113)) (justify left bottom))
-    )
-    (property "Footprint" "Capacitor_THT:C_Radial_D5.0mm_H11.0mm_P2.00mm" (at 274.32 46.355 0)
-      (effects (font (size 1.27 1.27)) hide)
-    )
-    (property "Datasheet" "" (at 274.32 46.355 0)
-      (effects (font (size 1.27 1.27)) hide)
-    )
-    (pin "1")
-    (pin "2")
-    (instances
-      (project "fieldRadio"
-        (path "/a1d1b2b0-2f27-4dc0-94ba-bb0e02933617/de17e96d-acc8-4488-9767-c0e10e15a863"
-          (reference "C52") (unit 1)
-        )
-      )
-      (project ""
-        (path "/c58960d9-4cac-4036-ad2e-1aef26946dae"
-          (reference "C9") (unit 1)
-        )
-      )
-      (project "powerAmp"
-        (path "/c63d077a-bb30-4740-8b96-a434a85a3a02"
-          (reference "C9") (unit 1)
-        )
-      )
-    )
-  )
   (symbol (lib_id "Device:Q_Dual_NMOS_S1G1S2G2D2D2D1D1") (at 196.85 178.435 0) (mirror x) (unit 2)
     (in_bom yes) (on_board yes) (dnp no)
@@
       (effects (font (size 1.27 1.27)) (justify left))
     )
-    (property "Footprint" "Transformer_THT:Autotransformer_Toroid_1Tap_Horizontal_D14.0mm_Amidon-T50" (at 218.44 167.005 0)
+    (property "Footprint" "Transformer_THT:Transformer_Toroid_Horizontal_D14.0mm_Amidon-T50" (at 218.44 167.005 0)
       (effects (font (size 1.27 1.27)) hide)
     )
@@
       (effects (font (size 1.27 1.27)) hide)
     )
+    (property "Mouser Part Number" "" (at 218.44 167.005 0)
+      (effects (font (size 1.27 1.27)) hide)
+    )
