File: fieldRadio/qsd.kicad_sch (KiCad schematic)
At the start: 41 parts, among them IC3 SN74LVC1G04DBVT, IC4 SN74AUP2G79DCUR, IC5 TS5A23157, IC6 SN74CBTLV3253, IC7 INA821ID, IC8 INA821ID, Q20 J309, T2 T50-TRIFILAR, U9 MCP1802x-xx02xOT

Commit message: Refine Placement 2
Finish refining block placement; ready for initial routing work.
Parts:
- removed C152: 0.1uF, Capacitor_SMD:C_0603_1608Metric_Pad1.08x0.95mm_HandSolder, symbol qsd_revB-eagle-import:CAP0603-CAP
- removed R142: 10k, Resistor_SMD:R_0603_1608Metric_Pad0.98x0.95mm_HandSolder, symbol qsd_revB-eagle-import:RESISTOR0603-RES
Changed lines of the file:
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@@
   (junction (at 269.24 96.52) (diameter 0) (color 0 0 0 0)
   )
-  (junction (at 177.8 160.02) (diameter 0) (color 0 0 0 0)
-  )
   (junction (at 193.04 81.28) (diameter 0) (color 0 0 0 0)
   )
@@
   (junction (at 274.32 78.74) (diameter 0) (color 0 0 0 0)
   )
-  (junction (at 403.86 45.72) (diameter 0) (color 0 0 0 0)
-  )
   (junction (at 295.91 96.52) (diameter 0) (color 0 0 0 0)
   )
@@
   (junction (at 210.82 180.34) (diameter 0) (color 0 0 0 0)
   )
-  (junction (at 378.46 45.72) (diameter 0) (color 0 0 0 0)
-  )
   (junction (at 378.46 88.9) (diameter 0) (color 0 0 0 0)
   )
@@
   (junction (at 149.86 137.16) (diameter 0) (color 0 0 0 0)
   )
-  (junction (at 187.96 180.34) (diameter 0) (color 0 0 0 0)
-  )
   (junction (at 251.46 144.78) (diameter 0) (color 0 0 0 0)
   )
@@
     (stroke (width 0) (type default))
   )
-  (wire (pts (xy 177.8 160.02) (xy 177.8 203.2))
-    (stroke (width 0) (type default))
-  )
-  (wire (pts (xy 378.46 38.1) (xy 378.46 45.72))
+  (wire (pts (xy 177.8 154.94) (xy 177.8 203.2))
     (stroke (width 0) (type default))
   )
@@
     (stroke (width 0) (type default))
   )
-  (wire (pts (xy 187.96 175.26) (xy 187.96 180.34))
-    (stroke (width 0) (type default))
-  )
   (wire (pts (xy 271.78 99.06) (xy 271.78 107.95))
     (stroke (width 0) (type default))
   )
-  (wire (pts (xy 210.82 180.34) (xy 187.96 180.34))
-    (stroke (width 0) (type default))
-  )
   (wire (pts (xy 149.86 127) (xy 76.2 127))
     (stroke (width 0) (type default))
@@
     (stroke (width 0) (type default))
   )
-  (wire (pts (xy 378.46 45.72) (xy 386.08 45.72))
-    (stroke (width 0) (type default))
-  )
   (wire (pts (xy 381 105.41) (xy 381 76.2))
     (stroke (width 0) (type default))
@@
     (stroke (width 0) (type default))
   )
-  (wire (pts (xy 177.8 154.94) (xy 177.8 160.02))
-    (stroke (width 0) (type default))
-  )
   (wire (pts (xy 226.06 127) (xy 251.46 127))
     (stroke (width 0) (type default))
@@
     (stroke (width 0) (type default))
   )
-  (wire (pts (xy 403.86 38.1) (xy 403.86 45.72))
-    (stroke (width 0) (type default))
-  )
   (wire (pts (xy 154.94 144.78) (xy 154.94 129.54))
     (stroke (width 0) (type default))
@@
     (stroke (width 0) (type default))
   )
-  (wire (pts (xy 393.7 45.72) (xy 403.86 45.72))
-    (stroke (width 0) (type default))
-  )
   (wire (pts (xy 271.78 107.95) (xy 284.48 107.95))
     (stroke (width 0) (type default))
@@
     (stroke (width 0) (type default))
   )
-  (wire (pts (xy 187.96 160.02) (xy 177.8 160.02))
-    (stroke (width 0) (type default))
-  )
   (wire (pts (xy 147.32 139.7) (xy 152.4 139.7))
     (stroke (width 0) (type default))
@@
     (stroke (width 0) (type default))
   )
-  (wire (pts (xy 187.96 165.1) (xy 187.96 160.02))
-    (stroke (width 0) (type default))
-  )
   (wire (pts (xy 264.16 127) (xy 251.46 127))
     (stroke (width 0) (type default))
@@
     (stroke (width 0) (type default))
   )
-  (wire (pts (xy 187.96 180.34) (xy 160.02 180.34))
+  (wire (pts (xy 160.02 180.34) (xy 210.82 180.34))
     (stroke (width 0) (type default))
   )
@@
     (stroke (width 0) (type default))
   )
-  (wire (pts (xy 378.46 45.72) (xy 378.46 71.12))
+  (wire (pts (xy 378.46 38.1) (xy 378.46 71.12))
     (stroke (width 0) (type default))
   )
@@
     (stroke (width 0) (type default))
   )
-  (wire (pts (xy 403.86 45.72) (xy 403.86 48.26))
+  (wire (pts (xy 403.86 38.1) (xy 403.86 48.26))
     (stroke (width 0) (type default))
   )
@@
         (path "/f12afe60-319a-4dbd-9291-4cc8914dd5dd"
           (reference "C13") (unit 1)
-        )
-      )
-    )
-  )
-  (symbol (lib_id "qsd_revB-eagle-import:RESISTOR0603-RES") (at 187.96 170.18 90) (unit 1)
-    (in_bom yes) (on_board yes) (dnp no)
-    (property "Reference" "R142" (at 195.072 168.1226 90)
-      (effects (font (size 1.778 1.5113)) (justify left bottom))
-    )
-    (property "Value" "10k" (at 195.58 170.688 90)
-      (effects (font (size 1.778 1.5113)) (justify left bottom))
-    )
-    (property "Footprint" "Resistor_SMD:R_0603_1608Metric_Pad0.98x0.95mm_HandSolder" (at 187.96 170.18 0)
-      (effects (font (size 1.27 1.27)) hide)
-    )
-    (property "Datasheet" "" (at 187.96 170.18 0)
-      (effects (font (size 1.27 1.27)) hide)
-    )
-    (pin "1")
-    (pin "2")
-    (instances
-      (project "fieldRadio"
-        (path "/a1d1b2b0-2f27-4dc0-94ba-bb0e02933617/b9a43a44-ac26-41be-aaf6-05c85180cb06"
-          (reference "R142") (unit 1)
-        )
-      )
-      (project "qsd_revC"
-        (path "/f12afe60-319a-4dbd-9291-4cc8914dd5dd"
-          (reference "R10") (unit 1)
         )
       )
@@
         )
       )
-    )
-  )
-  (symbol (lib_id "qsd_revB-eagle-import:CAP0603-CAP") (at 388.62 45.72 270) (unit 1)
-    (in_bom yes) (on_board yes) (dnp no)
-    (property "Reference" "C152" (at 383.286 45.085 90)
-      (effects (font (size 1.778 1.5113)) (justify left bottom))
-    )
-    (property "Value" "0.1uF" (at 392.176 45.085 90)
-      (effects (font (size 1.778 1.5113)) (justify left bottom))
-    )
-    (property "Footprint" "Capacitor_SMD:C_0603_1608Metric_Pad1.08x0.95mm_HandSolder" (at 388.62 45.72 0)
-      (effects (font (size 1.27 1.27)) hide)
-    )
-    (property "Datasheet" "" (at 388.62 45.72 0)
-      (effects (font (size 1.27 1.27)) hide)
-    )
-    (pin "1")
-    (pin "2")
-    (instances
-      (project "fieldRadio"
-        (path "/a1d1b2b0-2f27-4dc0-94ba-bb0e02933617/b9a43a44-ac26-41be-aaf6-05c85180cb06"
-          (reference "C152") (unit 1)
-        )
-      )
-      (project "qsd_revC"
-        (path "/f12afe60-319a-4dbd-9291-4cc8914dd5dd"
-          (reference "C20") (unit 1)
-        )
-      )
