File: fieldRadio_1.1/fieldRadio_1.1.kicad_sch (KiCad schematic)
At the start: 11 parts, among them J1 Conn_01x02, J18 Conn_01x16, J2 Conn_01x02, J3 Conn_01x03, J4 AudioJack2_Switch, J5 AudioJack3_Switch, J6 AudioJack2_Switch, J7 Conn_01x04, J8 Conn_01x12

Commit message: Rev 1.1 layout update
layout update routing and placement
Parts:
- J1, J2: footprint (none) -> Connector_PinHeader_2.54mm:PinHeader_1x02_P2.54mm_Vertical
- J18: footprint (none) -> Connector_PinHeader_2.54mm:PinHeader_1x16_P2.54mm_Vertical
- J8: footprint (none) -> Connector_PinHeader_2.54mm:PinHeader_1x12_P2.54mm_Vertical
Changed lines of the file:
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@@
       (effects (font (size 1.27 1.27)) (justify left))
     )
-    (property "Footprint" "" (at 265.43 79.375 0)
+    (property "Footprint" "Connector_PinHeader_2.54mm:PinHeader_1x12_P2.54mm_Vertical" (at 265.43 79.375 0)
       (effects (font (size 1.27 1.27)) hide)
     )
     (property "Datasheet" "~" (at 265.43 79.375 0)
+      (effects (font (size 1.27 1.27)) hide)
+    )
+    (property "Mouser Part Number" "" (at 265.43 79.375 0)
       (effects (font (size 1.27 1.27)) hide)
     )
@@
       (effects (font (size 1.27 1.27)) (justify left))
     )
-    (property "Footprint" "" (at 274.955 118.11 0)
+    (property "Footprint" "Connector_PinHeader_2.54mm:PinHeader_1x16_P2.54mm_Vertical" (at 274.955 118.11 0)
       (effects (font (size 1.27 1.27)) hide)
     )
     (property "Datasheet" "~" (at 274.955 118.11 0)
+      (effects (font (size 1.27 1.27)) hide)
+    )
+    (property "Mouser Part Number" "" (at 274.955 118.11 0)
       (effects (font (size 1.27 1.27)) hide)
     )
@@
       (effects (font (size 1.27 1.27)) (justify left))
     )
-    (property "Footprint" "" (at 38.1 22.86 0)
+    (property "Footprint" "Connector_PinHeader_2.54mm:PinHeader_1x02_P2.54mm_Vertical" (at 38.1 22.86 0)
       (effects (font (size 1.27 1.27)) hide)
     )
@@
       (effects (font (size 1.27 1.27)) hide)
     )
+    (property "Mouser Part Number" "" (at 38.1 22.86 0)
+      (effects (font (size 1.27 1.27)) hide)
+    )
     (pin "2")
     (pin "1")
@@
       (effects (font (size 1.27 1.27)) (justify left))
     )
-    (property "Footprint" "" (at 26.416 175.26 0)
+    (property "Footprint" "Connector_PinHeader_2.54mm:PinHeader_1x02_P2.54mm_Vertical" (at 26.416 175.26 0)
       (effects (font (size 1.27 1.27)) hide)
     )
@@
       (effects (font (size 1.27 1.27)) hide)
     )
+    (property "Mouser Part Number" "" (at 26.416 175.26 0)
+      (effects (font (size 1.27 1.27)) hide)
+    )

Commit message: Button Board
added button board
Parts:
- added J12: Conn_01x02, Connector_PinHeader_2.54mm:PinHeader_1x02_P2.54mm_Vertical, symbol Connector_Generic:Conn_01x02
Connections:
- net at J6.SN: now also J12.2 (Pin_2)
- net at J6.TN: now also J12.1 (Pin_1)
- no-connect marks 15 -> 13
Other:
- note added: "For connection to internal speaker"
Changed lines of the file:
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@@
   (no_connect (at 152.4 180.34))
   (no_connect (at 152.4 185.42))
-  (no_connect (at 252.73 39.37))
   (no_connect (at 269.875 115.57))
   (no_connect (at 269.875 123.19))
@@
   (no_connect (at 154.305 168.91))
   (no_connect (at 167.64 144.78))
-  (no_connect (at 252.73 34.29))
   (no_connect (at 269.875 118.11))
   (no_connect (at 154.305 173.99))
@@
     (stroke (width 0) (type default))
   )
+  (wire (pts (xy 252.73 20.828) (xy 252.73 34.29))
+    (stroke (width 0) (type default))
+  )
   (bus (pts (xy 243.205 71.755) (xy 243.205 74.295))
     (stroke (width 0) (type default))
@@
     (stroke (width 0) (type default))
   )
+  (wire (pts (xy 247.396 39.37) (xy 247.396 23.368))
+    (stroke (width 0) (type default))
+  )
   (wire (pts (xy 167.64 102.87) (xy 171.45 102.87))
     (stroke (width 0) (type default))
@@
     (stroke (width 0) (type default))
   )
+  (wire (pts (xy 252.73 39.37) (xy 247.396 39.37))
+    (stroke (width 0) (type default))
+  )
   (wire (pts (xy 256.54 128.27) (xy 269.875 128.27))
     (stroke (width 0) (type default))
@@
     (stroke (width 0) (type default))
   )
+  (wire (pts (xy 246.38 20.828) (xy 252.73 20.828))
+    (stroke (width 0) (type default))
+  )
   (wire (pts (xy 226.06 88.265) (xy 212.09 88.265))
     (stroke (width 0) (type default))
@@
   )
   (bus (pts (xy 173.355 168.91) (xy 173.355 180.34))
+    (stroke (width 0) (type default))
+  )
+  (wire (pts (xy 247.396 23.368) (xy 246.38 23.368))
     (stroke (width 0) (type default))
   )
@@
   (text "E" (at 278.765 114.935 0)
     (effects (font (size 1.778 1.5113)) (justify right bottom))
+  )
+  (text "For connection\nto internal\nspeaker" (at 215.9 25.654 0)
+    (effects (font (size 1.27 1.27)) (justify left bottom))
   )
   (text "DB2" (at 281.305 122.555 0)
@@
         )
       )
+    )
+  )
+  (symbol (lib_id "Connector_Generic:Conn_01x02") (at 241.3 20.828 0) (mirror y) (unit 1)
+    (in_bom yes) (on_board yes) (dnp no)
+    (property "Reference" "J12" (at 238.76 20.828 0)
+      (effects (font (size 1.27 1.27)) (justify left))
+    )
+    (property "Value" "Conn_01x02" (at 238.76 23.368 0)
+      (effects (font (size 1.27 1.27)) (justify left))
+    )
+    (property "Footprint" "Connector_PinHeader_2.54mm:PinHeader_1x02_P2.54mm_Vertical" (at 241.3 20.828 0)
+      (effects (font (size 1.27 1.27)) hide)
+    )
+    (property "Datasheet" "~" (at 241.3 20.828 0)
+      (effects (font (size 1.27 1.27)) hide)
+    )
+    (property "Mouser Part Number" "" (at 241.3 20.828 0)
+      (effects (font (size 1.27 1.27)) hide)
+    )
+    (pin "2")
+    (pin "1")
+    (instances
+      (project "fieldRadio_1.1"
+        (path "/a1d1b2b0-2f27-4dc0-94ba-bb0e02933617"
+          (reference "J12") (unit 1)
+        )
+      )
