File: fieldRadio_1.1/TRSwitch.kicad_sch (KiCad schematic)
At the start: 36 parts, among them Q1 MMBT3904, Q2 MMBT3904, Q3 PMV240SP, Q5 MMBT3904, Q6 PMV240SP, Q7 BSS123

Commit message: work on button selector schematic
Parts:
- renumbered C1 to C3, C2 to C4, C4 to C5, C5 to C6, C3 to C7, C7 to C8, C6 to C9, Q5 to Q4, Q6 to Q5, Q7 to Q6, R13 to R10, R10 to R11, R11 to R12, R9 to R13, R12 to R7, R7 to R8, R8 to R9
