File: QEX_PowerAmp_Experiment/QEX_PowerAmp_Experiment.kicad_pcb (KiCad board)
At the start: 4 copper layers, 87 x 74 mm, 73 parts, among them J1 Key In, J10 Conn_01x02, J11 SMA, J12 Conn_01x02, J2 Key In, J3 Conn_01x02, J4 Conn_01x02, J5 SMA, J6 Conn_01x02, J7 Conn_01x02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

Commit message: Refining layout
Parts:
- moved R3 0.29 mm to (148.0, 75.5)
- moved C1 0.25 mm to (144.0, 74.5)
- moved C11 0.25 mm to (152.5, 70.0)
- moved C5 0.25 mm to (152.0, 74.5)
- moved U2 0.25 mm to (148.0, 70.0)
- moved J2 0.22 mm to (106.5, 75.0)
Routing:
- net GND: track 67.8 -> 68.6 mm
Other:
- rule pad_to_mask_clearance: 0 -> 0.1
Changed lines of the file:
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@@
 			(dielectric_constraints no)
 		)
-		(pad_to_mask_clearance 0)
+		(pad_to_mask_clearance 0.1)
+		(solder_mask_min_width 0.1)
 		(allow_soldermask_bridges_in_footprints no)
 		(tenting front back)
@@
 	(footprint "PCM_JLCPCB:C_0603"
 		(layer "F.Cu")
-		(at 152.1 74.725 90)
+		(at 152 74.5 90)
 		(descr "Capacitor SMD 0603 (1608 Metric), square (rectangular) end terminal, IPC_7351 nominal, (Body size source: IPC-SM-782 page 76, https://www.pcb-3d.com/wordpress/wp-content/uploads/ipc-sm-782a_amendment_1_and_2.pdf), generated with kicad-footprint-generator")
 		(tags "capacitor")
@@
 	(footprint "Connector_PinHeader_2.54mm:PinHeader_1x02_P2.54mm_Vertical"
 		(layer "F.Cu")
-		(at 106.5 75.225)
+		(at 106.5 75)
 		(descr "Through hole straight pin header, 1x02, 2.54mm pitch, single row")
 		(tags "Through hole pin header THT 1x02 2.54mm single row")
@@
 	(footprint "Resistor_SMD:R_0805_2012Metric_Pad1.20x1.40mm_HandSolder"
 		(layer "F.Cu")
-		(at 148.1 75.225)
+		(at 148 75.5)
 		(descr "Resistor SMD 0805 (2012 Metric), square (rectangular) end terminal, IPC-7351 nominal with elongated pad for handsoldering. (Body size source: IPC-SM-782 page 72, https://www.pcb-3d.com/wordpress/wp-content/uploads/ipc-sm-782a_amendment_1_and_2.pdf), generated with kicad-footprint-generator")
 		(tags "resistor handsolder")
@@
 	(footprint "PCM_JLCPCB:C_0603"
 		(layer "F.Cu")
-		(at 144.1 74.725 90)
+		(at 144 74.5 90)
 		(descr "Capacitor SMD 0603 (1608 Metric), square (rectangular) end terminal, IPC_7351 nominal, (Body size source: IPC-SM-782 page 76, https://www.pcb-3d.com/wordpress/wp-content/uploads/ipc-sm-782a_amendment_1_and_2.pdf), generated with kicad-footprint-generator")
 		(tags "capacitor")
@@
 	(footprint "PCM_JLCPCB:C_0603"
 		(layer "F.Cu")
-		(at 152.6 70.225)
+		(at 152.5 70)
 		(descr "Capacitor SMD 0603 (1608 Metric), square (rectangular) end terminal, IPC_7351 nominal, (Body size source: IPC-SM-782 page 76, https://www.pcb-3d.com/wordpress/wp-content/uploads/ipc-sm-782a_amendment_1_and_2.pdf), generated with kicad-footprint-generator")
 		(tags "capacitor")
@@
 	(footprint "Package_TO_SOT_SMD:SOT-23-5"
 		(layer "F.Cu")
-		(at 148.1 70.225)
+		(at 148 70)
 		(descr "SOT, 5 Pin (JEDEC MO-178 Var AA https://www.jedec.org/document_search?search_api_views_fulltext=MO-178), generated with kicad-footprint-generator ipc_gullwing_generator.py")
 		(tags "SOT TO_SOT_SMD")
@@
 	)
 	(segment
-		(start 146.9625 70.225)
-		(end 145.225 70.225)
-		(width 0.5)
-		(layer "F.Cu")
-		(net 1)
-	)
-	(segment
 		(start 128.05 83.45)
 		(end 128 83.5)
@@
 	)
 	(segment
+		(start 144.1 73.945)
+		(end 142.055 73.945)
+		(width 0.5)
+		(layer "F.Cu")
+		(net 1)
+	)
+	(segment
 		(start 130.45 105)
 		(end 132.5 105)
@@
 	)
 	(segment
+		(start 142.055 73.945)
+		(end 142 74)
+		(width 0.5)
+		(layer "F.Cu")
+		(net 1)
+	)
+	(segment
 		(start 130.45 102.5)
 		(end 132.5 102.5)
@@
 	)
 	(segment
-		(start 142.555 73.945)
-		(end 142.5 74)
-		(width 0.5)
-		(layer "F.Cu")
-		(net 1)
-	)
-	(segment
 		(start 118.22 61.5)
 		(end 116.5 61.5)
@@
 	)
 	(segment
+		(start 146.8625 70)
+		(end 144.5 70)
+		(width 0.5)
+		(layer "F.Cu")
+		(net 1)
+	)
+	(segment
 		(start 122.95 126)
 		(end 125 126)
@@
 	)
 	(segment
-		(start 144.1 73.945)
-		(end 142.555 73.945)
-		(width 0.5)
-		(layer "F.Cu")
-		(net 1)
-	)
-	(segment
 		(start 133.023196 83.473196)
 		(end 133 83.45)
@@
 	)
 	(segment
-		(start 145.225 70.225)
-		(end 145 70)
-		(width 0.5)
-		(layer "F.Cu")
-		(net 1)
-	)
-	(segment
 		(start 137.78 82.72)
 		(end 138.5 82)
@@
 	)
 	(via
-		(at 145 70)
+		(at 144.5 70)
 		(size 1.2)
 		(drill 0.6)
@@
 	)
 	(via
-		(at 142.5 74)
+		(at 142 74)
 		(size 1.2)
 		(drill 0.6)
@@
 	)
 	(segment
-		(start 150.87 69.275)
-		(end 151.82 70.225)
-		(width 0.5)
-		(layer "F.Cu")
-		(net 5)
-	)
-	(segment
 		(start 153.595 72)
 		(end 154 72)
@@
 	)
 	(segment
+		(start 149.1375 69.05)
+		(end 149.3625 69.275)
+		(width 0.5)
+		(layer "F.Cu")
+		(net 5)
+	)
+	(segment
 		(start 124.15 108.65)
 		(end 123 107.5)
@@
 	)
 	(segment
+		(start 150.87 69.275)
+		(end 151.82 70.225)
+		(width 0.5)
+		(layer "F.Cu")
+		(net 5)
+	)
+	(segment
 		(start 120.45 114.17)
 		(end 120.28 114)
@@
 	)
 	(segment
+		(start 149.3625 69.275)
+		(end 150.87 69.275)
+		(width 0.5)
+		(layer "F.Cu")
+		(net 5)
+	)
+	(segment
 		(start 116.55 122.95)
 		(end 116 123.5)
@@
 	)
 	(segment
-		(start 149.2375 69.275)
-		(end 150.87 69.275)
-		(width 0.5)
-		(layer "F.Cu")
-		(net 5)
-	)
-	(segment
 		(start 124.55 108.65)
 		(end 124.15 108.65)
@@
 	)
 	(segment
-		(start 149.2375 67)
-		(end 166 67)
+		(start 170.5 65)
+		(end 171.225 64.275)
 		(width 0.5)
 		(layer "F.Cu")
@@
 	)
 	(segment
-		(start 170.5 65)
-		(end 171.225 64.275)
+		(start 168 65)
+		(end 170.5 65)
 		(width 0.5)
 		(layer "F.Cu")
@@
 	)
 	(segment
-		(start 171.225 64.275)
-		(end 171.225 59)
+		(start 149.2375 67)
+		(end 166 67)
 		(width 0.5)
 		(layer "F.Cu")
@@
 	)
 	(segment
-		(start 146.9625 69.275)
+		(start 147.1875 69.05)
 		(end 149.2375 67)
 		(width 0.5)
@@
 	)
 	(segment
-		(start 168 65)
-		(end 170.5 65)
+		(start 146.8625 69.05)
+		(end 147.1875 69.05)
+		(width 0.5)
+		(layer "F.Cu")
+		(net 26)
+	)
+	(segment
+		(start 171.225 64.275)
+		(end 171.225 59)
 		(width 0.5)
 		(layer "F.Cu")
@@
 	)
 	(segment
-		(start 144.1 75.505)
-		(end 146.82 75.505)
-		(width 1)
-		(layer "F.Cu")
-		(net 41)
-	)
-	(segment
 		(start 147.1 75.225)
 		(end 147.1 78.6)
@@
 	)
 	(segment
+		(start 147.1 75.225)
+		(end 144.055 75.225)
+		(width 0.5)
+		(layer "F.Cu")
+		(net 41)
+	)
+	(segment
+		(start 144.055 75.225)
+		(end 144 75.28)
+		(width 0.5)
+		(layer "F.Cu")
+		(net 41)
+	)
+	(segment
 		(start 177.95 107.5)
 		(end 179 106.45)
@@
 		(min_thickness 0.25)
 		(filled_areas_thickness no)
-		(fill yes
+		(fill
 			(thermal_gap 0.5)
 			(thermal_bridge_width 1)
@@
 		(min_thickness 0.25)
 		(filled_areas_thickness no)
-		(fill yes
+		(fill
 			(thermal_gap 0.5)
 			(thermal_bridge_width 1)
@@
 		(min_thickness 0.25)
 		(filled_areas_thickness no)
-		(fill yes
+		(fill
 			(thermal_gap 0.5)
 			(thermal_bridge_width 1)
@@
 		(min_thickness 0.2)
 		(filled_areas_thickness no)
-		(fill yes
+		(fill
 			(thermal_gap 0.5)
 			(thermal_bridge_width 1)
@@
 		(min_thickness 0.25)
 		(filled_areas_thickness no)
-		(fill yes
+		(fill
 			(thermal_gap 0.5)
 			(thermal_bridge_width 1)
@@
 		(min_thickness 0.25)
 		(filled_areas_thickness no)
-		(fill yes
+		(fill
 			(thermal_gap 0.5)
 			(thermal_bridge_width 1)

Commit message: Final PCB and BOM changes before tapeout
Parts:
- moved R16 1.80 mm to (134.0, 60.0)
- moved C7 0.25 mm to (121.8, 126.0)
Connections:
- net Net-(J3-Pin_1) renamed /pwr-in
Routing:
- net GND: track 68.6 -> 73.6 mm
- net Net-(U8D--): track 7.06 -> 5.14 mm
- net /k4: track 14.2 -> 13.6 mm
Other:
- rule pad_to_mask_clearance: 0.1 -> 0
- board text added: "+"
