File: fieldRadio_1.2/lpf_relayTest/lpf_relayTest.kicad_pcb (KiCad board)
At the start: 4 copper layers, 108 x 82 mm, 71 parts, among them J1 Conn_Coaxial_Small, J2 Conn_Coaxial_Small, J3 Conn_Coaxial_Small, J4 Conn_Coaxial_Small, J5 Conn_01x02, J6 Conn_01x02, J7 Conn_01x02, J8 Conn_01x02, K1 G6SU-2, K2 G6SU-2, K3 G6SU-2, K4 G6SU-2, K5 G6SU-2, K6 G6SU-2, U1 74HC595, U2 74ACT244, U3 74ACT125

Commit message: Updates to tonedecoder, swrpr. field radio 1.1
Parts:
- L12: value 560pF -> 560nF
