File: fieldRadio_1.2/audioFilters.kicad_sch (KiCad schematic)
At the start: 41 parts, among them U14 TS5A3159ADBVR, U15 TS5A3159ADBVR, U18 OPA1679, U6 OPA1679

Commit message: adding jlcpcb part numbers to schematics
Parts:
- removed RV1: 1K, Potentiometer_THT:Potentiometer_Bourns_3296W_Vertical, symbol Device:R_Potentiometer_US
- added R19: 300Ω, PCM_JLCPCB:R_0603, symbol PCM_JLCPCB-Resistors:0603,300Ω
- added R20: 1.2kΩ, PCM_JLCPCB:R_0603, symbol PCM_JLCPCB-Resistors:0603,1.2kΩ
- added R21: 3.3kΩ, PCM_JLCPCB:R_0603, symbol PCM_JLCPCB-Resistors:0603,3.3kΩ
- added R25: 18kΩ, PCM_JLCPCB:R_0603, symbol PCM_JLCPCB-Resistors:0603,18kΩ
- added RV4: 1K pot, Potentiometer_THT:Potentiometer_Bourns_3296W_Vertical, symbol Device:R_Potentiometer_US
- C57, C65: footprint Capacitor_THT:CP_Radial_D5.0mm_P2.50mm -> PCM_JLCPCB:C_0805; symbol Device:C_Polarized_US -> PCM_JLCPCB-Capacitors:0805,4.7uF; Attrition Qty (none) -> 10; Capacitance (none) -> 4.7uF; Category (none) -> Capacitors,Multilayer Ceramic Capacitors MLCC - SMD/SMT; Class (none) -> Basic Component; LCSC (none) -> C1779; Manufacturer (none) -> Samsung Electro-Mechanics; Minimum Qty (none) -> 20; Part (none) -> CL21A475KAQNNNE; Price (none) -> 0.015USD; Process (none) -> SMT; Stock (none) -> 1824431; Temperature Coefficient (none) -> X5R; Tolerance (none) -> ±10%; Voltage Rated (none) -> 25V
- C58, C59, C62, C63, C64: footprint Capacitor_SMD:C_0603_1608Metric_Pad1.08x0.95mm_HandSolder -> PCM_JLCPCB:C_0603; symbol Device:C -> PCM_JLCPCB-Capacitors:0603,100nF; Attrition Qty (none) -> 10; Capacitance (none) -> 100nF; Category (none) -> Capacitors,Multilayer Ceramic Capacitors MLCC - SMD/SMT; Class (none) -> Basic Component; LCSC (none) -> C14663; Manufacturer (none) -> YAGEO; Minimum Qty (none) -> 20; Part (none) -> CC0603KRX7R9BB104; Price (none) -> 0.006USD; Process (none) -> SMT; Stock (none) -> 70324515; Temperature Coefficient (none) -> X7R; Tolerance (none) -> ±10%; Voltage Rated (none) -> 50V
- C60, C61, C67, C68, C69, C70: value 0.01u -> 10nF; footprint Capacitor_SMD:C_0603_1608Metric_Pad1.08x0.95mm_HandSolder -> PCM_JLCPCB:C_0603; symbol Device:C -> PCM_JLCPCB-Capacitors:0603,10nF; Attrition Qty (none) -> 10; Capacitance (none) -> 10nF; Category (none) -> Capacitors,Multilayer Ceramic Capacitors MLCC - SMD/SMT; Class (none) -> Basic Component; LCSC (none) -> C57112; Manufacturer (none) -> FH(Guangdong Fenghua Advanced Tech); Minimum Qty (none) -> 20; Part (none) -> 0603B103K500NT; Price (none) -> 0.005USD; Process (none) -> SMT; Stock (none) -> 5921160; Temperature Coefficient (none) -> X7R; Tolerance (none) -> ±10%; Voltage Rated (none) -> 50V
- R40: value 1.5K -> 1.5kΩ; footprint Resistor_SMD:R_0603_1608Metric_Pad0.98x0.95mm_HandSolder -> PCM_JLCPCB:R_0603; symbol Device:R_US -> PCM_JLCPCB-Resistors:0603,1.5kΩ; Attrition Qty (none) -> 10; Category (none) -> Resistors,Chip Resistor - Surface Mount; Class (none) -> Basic Component; LCSC (none) -> C22843; Manufacturer (none) -> UNI-ROYAL(Uniroyal Elec); Minimum Qty (none) -> 20; Operating Temperature Range (none) -> -55°C~+155°C; Overload Voltage (Max) (none) -> 75V; Part (none) -> 0603WAF1501T5E; Power(Watts) (none) -> 100mW; Price (none) -> 0.004USD; Process (none) -> SMT; Resistance (none) -> 1.5kΩ; Stock (none) -> 2582969; Temperature Coefficient (none) -> ±100ppm/°C; Tolerance (none) -> ±1%; Type (none) -> Thick Film Resistors
- R41, R43, R45, R46, R47, R48, R49, R51, R53, R54, R55, R57, R59, R60: value 10K -> 10kΩ; footprint Resistor_SMD:R_0603_1608Metric_Pad0.98x0.95mm_HandSolder -> PCM_JLCPCB:R_0603; symbol Device:R_US -> PCM_JLCPCB-Resistors:0603,10kΩ; Attrition Qty (none) -> 10; Category (none) -> Resistors,Chip Resistor - Surface Mount; Class (none) -> Basic Component; LCSC (none) -> C25804; Manufacturer (none) -> UNI-ROYAL(Uniroyal Elec); Minimum Qty (none) -> 20; Operating Temperature Range (none) -> -55°C~+155°C; Overload Voltage (Max) (none) -> 75V; Part (none) -> 0603WAF1002T5E; Power(Watts) (none) -> 100mW; Price (none) -> 0.004USD; Process (none) -> SMT; Resistance (none) -> 10kΩ; Stock (none) -> 51181774; Temperature Coefficient (none) -> ±100ppm/°C; Tolerance (none) -> ±1%; Type (none) -> Thick Film Resistors
- R42: value 200 -> 200Ω; footprint Resistor_SMD:R_0603_1608Metric_Pad0.98x0.95mm_HandSolder -> PCM_JLCPCB:R_0603; symbol Device:R_US -> PCM_JLCPCB-Resistors:0603,200Ω; Attrition Qty (none) -> 10; Category (none) -> Resistors,Chip Resistor - Surface Mount; Class (none) -> Basic Component; LCSC (none) -> C8218; Manufacturer (none) -> UNI-ROYAL(Uniroyal Elec); Minimum Qty (none) -> 20; Operating Temperature Range (none) -> -55°C~+155°C; Overload Voltage (Max) (none) -> 75V; Part (none) -> 0603WAF2000T5E; Power(Watts) (none) -> 100mW; Price (none) -> 0.004USD; Process (none) -> SMT; Resistance (none) -> 200Ω; Stock (none) -> 2444311; Temperature Coefficient (none) -> ±100ppm/°C; Tolerance (none) -> ±1%; Type (none) -> Thick Film Resistors
- R44: value 5.23K -> 5.1kΩ; footprint Resistor_SMD:R_0603_1608Metric_Pad0.98x0.95mm_HandSolder -> PCM_JLCPCB:R_0603; symbol Device:R_US -> PCM_JLCPCB-Resistors:0603,5.1kΩ; Attrition Qty (none) -> 10; Category (none) -> Resistors,Chip Resistor - Surface Mount; Class (none) -> Basic Component; LCSC (none) -> C23186; Manufacturer (none) -> UNI-ROYAL(Uniroyal Elec); Minimum Qty (none) -> 20; Operating Temperature Range (none) -> -55°C~+155°C; Overload Voltage (Max) (none) -> 75V; Part (none) -> 0603WAF5101T5E; Power(Watts) (none) -> 100mW; Price (none) -> 0.004USD; Process (none) -> SMT; Resistance (none) -> 5.1kΩ; Stock (none) -> 9223405; Temperature Coefficient (none) -> ±100ppm/°C; Tolerance (none) -> ±1%; Type (none) -> Thick Film Resistors
- R50: value 11.3K -> 11kΩ; footprint Resistor_SMD:R_0603_1608Metric_Pad0.98x0.95mm_HandSolder -> PCM_JLCPCB:R_0603; symbol Device:R_US -> PCM_JLCPCB-Resistors:0603,11kΩ; Attrition Qty (none) -> 10; Category (none) -> Resistors,Chip Resistor - Surface Mount; Class (none) -> Preferred Component; LCSC (none) -> C25950; Manufacturer (none) -> UNI-ROYAL(Uniroyal Elec); Minimum Qty (none) -> 20; Operating Temperature Range (none) -> -55°C~+155°C; Overload Voltage (Max) (none) -> 75V; Part (none) -> 0603WAF1102T5E; Power(Watts) (none) -> 100mW; Price (none) -> 0.004USD; Process (none) -> SMT; Resistance (none) -> 11kΩ; Stock (none) -> 332012; Temperature Coefficient (none) -> ±100ppm/°C; Tolerance (none) -> ±1%; Type (none) -> Thick Film Resistors
- R52: value 23.2K -> 20kΩ; footprint Resistor_SMD:R_0603_1608Metric_Pad0.98x0.95mm_HandSolder -> PCM_JLCPCB:R_0603; symbol Device:R_US -> PCM_JLCPCB-Resistors:0603,20kΩ; Attrition Qty (none) -> 10; Category (none) -> Resistors,Chip Resistor - Surface Mount; Class (none) -> Basic Component; LCSC (none) -> C4184; Manufacturer (none) -> UNI-ROYAL(Uniroyal Elec); Minimum Qty (none) -> 20; Operating Temperature Range (none) -> -55°C~+155°C; Overload Voltage (Max) (none) -> 75V; Part (none) -> 0603WAF2002T5E; Power(Watts) (none) -> 100mW; Price (none) -> 0.004USD; Process (none) -> SMT; Resistance (none) -> 20kΩ; Stock (none) -> 3333761; Temperature Coefficient (none) -> ±100ppm/°C; Tolerance (none) -> ±1%; Type (none) -> Thick Film Resistors
- R56: value 51.1K -> 51kΩ; footprint Resistor_SMD:R_0603_1608Metric_Pad0.98x0.95mm_HandSolder -> PCM_JLCPCB:R_0603; symbol Device:R_US -> PCM_JLCPCB-Resistors:0603,51kΩ; Attrition Qty (none) -> 10; Category (none) -> Resistors,Chip Resistor - Surface Mount; Class (none) -> Basic Component; LCSC (none) -> C23196; Manufacturer (none) -> UNI-ROYAL(Uniroyal Elec); Minimum Qty (none) -> 20; Operating Temperature Range (none) -> -55°C~+155°C; Overload Voltage (Max) (none) -> 75V; Part (none) -> 0603WAF5102T5E; Power(Watts) (none) -> 100mW; Price (none) -> 0.004USD; Process (none) -> SMT; Resistance (none) -> 51kΩ; Stock (none) -> 1964861; Temperature Coefficient (none) -> ±100ppm/°C; Tolerance (none) -> ±1%; Type (none) -> Thick Film Resistors
- R58: value 178K -> 160kΩ; footprint Resistor_SMD:R_0603_1608Metric_Pad0.98x0.95mm_HandSolder -> PCM_JLCPCB:R_0603; symbol Device:R_US -> PCM_JLCPCB-Resistors:0603,160kΩ; Attrition Qty (none) -> 10; Category (none) -> Resistors,Chip Resistor - Surface Mount; Class (none) -> Preferred Component; LCSC (none) -> C22813; Manufacturer (none) -> UNI-ROYAL(Uniroyal Elec); Minimum Qty (none) -> 20; Operating Temperature Range (none) -> -55°C~+155°C; Overload Voltage (Max) (none) -> 75V; Part (none) -> 0603WAF1603T5E; Power(Watts) (none) -> 100mW; Price (none) -> 0.004USD; Process (none) -> SMT; Resistance (none) -> 160kΩ; Stock (none) -> 66800; Temperature Coefficient (none) -> ±100ppm/°C; Tolerance (none) -> ±1%; Type (none) -> Thick Film Resistors
- R61, R62: value 1K -> 1kΩ; footprint Resistor_SMD:R_0603_1608Metric_Pad0.98x0.95mm_HandSolder -> PCM_JLCPCB:R_0603; symbol Device:R_US -> PCM_JLCPCB-Resistors:0603,1kΩ; Attrition Qty (none) -> 10; Category (none) -> Resistors,Chip Resistor - Surface Mount; Class (none) -> Basic Component; LCSC (none) -> C21190; Manufacturer (none) -> UNI-ROYAL(Uniroyal Elec); Minimum Qty (none) -> 20; Operating Temperature Range (none) -> -55°C~+155°C; Overload Voltage (Max) (none) -> 75V; Part (none) -> 0603WAF1001T5E; Power(Watts) (none) -> 100mW; Price (none) -> 0.004USD; Process (none) -> SMT; Resistance (none) -> 1kΩ; Stock (none) -> 27538425; Temperature Coefficient (none) -> ±100ppm/°C; Tolerance (none) -> ±1%; Type (none) -> Thick Film Resistors
- U14, U15: value TS5A3159ADBVR -> TS5A3159ADCK; footprint Package_TO_SOT_SMD:SOT-23-6 -> Package_TO_SOT_SMD:SOT-363_SC-70-6; symbol Analog_Switch:TS5A3159ADBVR -> Analog_Switch:TS5A3159ADCK; JLCPCB (none) -> C46388
- U18, U6: JLCPCB (none) -> C2878631
Connections:
- net Q: now also R20.1; no longer R44.1
- net at R61.2: now also RV4.1
- net at U18.10 (+): now also RV4.2
- net at R62.2: now also RV4.3
- net at R47.2, R51.1, U6.8: now also R21.1; no longer R52.1
- net at R46.2, R49.1, U6.1: now also R19.1; no longer R50.1
- net at R54.2, R57.1, U6.14: now also R25.1; no longer R58.1
- new net: R19.2, R50.1
- new net: R20.2, R44.1
- new net: R25.2, R58.1
- new net: R21.2, R52.1

Commit message: continued symbol property updates
Parts:
- RV4: now left out of the parts list
- U14, U15: LCSC (none) -> C46388
- U18, U6: LCSC (none) -> C2878631
Changed lines of the file:
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@@
 			)
 		)
+		(property "LCSC" "C2878631"
+			(at 200.66 149.86 0)
+			(hide yes)
+			(show_name no)
+			(do_not_autoplace no)
+			(effects
+				(font
+					(size 1.27 1.27)
+				)
+			)
+		)
 		(pin "11"
 		)
@@
 			)
 		)
+		(property "LCSC" "C2878631"
+			(at 256.54 66.04 0)
+			(hide yes)
+			(show_name no)
+			(do_not_autoplace no)
+			(effects
+				(font
+					(size 1.27 1.27)
+				)
+			)
+		)
 		(pin "11"
 		)
@@
 			)
 		)
+		(property "LCSC" "C2878631"
+			(at 170.18 175.26 0)
+			(hide yes)
+			(show_name no)
+			(do_not_autoplace no)
+			(effects
+				(font
+					(size 1.27 1.27)
+				)
+			)
+		)
 		(pin "11"
 		)
@@
 			)
 		)
+		(property "LCSC" "C2878631"
+			(at 257.81 107.95 0)
+			(hide yes)
+			(show_name no)
+			(do_not_autoplace no)
+			(effects
+				(font
+					(size 1.27 1.27)
+				)
+			)
+		)
 		(pin "11"
 		)
@@
 		(body_style 1)
 		(exclude_from_sim no)
-		(in_bom yes)
+		(in_bom no)
 		(on_board yes)
 		(in_pos_files yes)
@@
 			)
 		)
+		(property "LCSC" "C2878631"
+			(at 153.67 66.04 0)
+			(hide yes)
+			(show_name no)
+			(do_not_autoplace no)
+			(effects
+				(font
+					(size 1.27 1.27)
+				)
+			)
+		)
 		(pin "13"
 		)
@@
 			)
 		)
+		(property "LCSC" "C2878631"
+			(at 125.73 175.26 0)
+			(hide yes)
+			(show_name no)
+			(do_not_autoplace no)
+			(effects
+				(font
+					(size 1.27 1.27)
+				)
+			)
+		)
 		(pin "13"
 		)
@@
 			)
 		)
+		(property "LCSC" "C46388"
+			(at 355.6 82.55 0)
+			(hide yes)
+			(show_name no)
+			(do_not_autoplace no)
+			(effects
+				(font
+					(size 1.27 1.27)
+				)
+			)
+		)
 		(pin "6"
 		)
@@
 			)
 		)
+		(property "LCSC" "C46388"
+			(at 189.23 177.8 0)
+			(hide yes)
+			(show_name no)
+			(do_not_autoplace no)
+			(effects
+				(font
+					(size 1.27 1.27)
+				)
+			)
+		)
 		(pin "6"
 		)
@@
 			)
 		)
+		(property "LCSC" "C2878631"
+			(at 204.47 107.95 0)
+			(hide yes)
+			(show_name no)
+			(do_not_autoplace no)
+			(effects
+				(font
+					(size 1.27 1.27)
+				)
+			)
+		)
 		(pin "13"
 		)
@@
 			)
 		)
+		(property "LCSC" "C2878631"
+			(at 204.47 66.04 0)
+			(hide yes)
+			(show_name no)
+			(do_not_autoplace no)
+			(effects
+				(font
+					(size 1.27 1.27)
+				)
+			)
+		)
 		(pin "13"
 		)
@@
 			)
 		)
+		(property "LCSC" "C2878631"
+			(at 308.61 87.63 0)
+			(hide yes)
+			(show_name no)
+			(do_not_autoplace no)
+			(effects
+				(font
+					(size 1.27 1.27)
+				)
+			)
+		)
 		(pin "11"
 		)
@@
 			(at 154.94 107.95 0)
 			(hide yes)
+			(show_name no)
+			(do_not_autoplace no)
+			(effects
+				(font
+					(size 1.27 1.27)
+				)
+			)
+		)
+		(property "LCSC" "C2878631"
+			(at 154.94 107.95 0)
+			(hide yes)

Commit message: ready to start layout
Parts:
- U18, U6: footprint (none) -> Package_SO:SOIC-14_3.9x8.7mm_P1.27mm
Changed lines of the file:
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@@
 			)
 		)
-		(property "Footprint" ""
+		(property "Footprint" "Package_SO:SOIC-14_3.9x8.7mm_P1.27mm"
 			(at 199.39 147.32 0)
 			(hide yes)
@@
 			)
 		)
-		(property "Footprint" ""
+		(property "Footprint" "Package_SO:SOIC-14_3.9x8.7mm_P1.27mm"
 			(at 255.27 68.58 0)
 			(hide yes)
@@
 			)
 		)
-		(property "Footprint" ""
+		(property "Footprint" "Package_SO:SOIC-14_3.9x8.7mm_P1.27mm"
 			(at 168.91 172.72 0)
 			(hide yes)
@@
 			)
 		)
-		(property "Footprint" ""
+		(property "Footprint" "Package_SO:SOIC-14_3.9x8.7mm_P1.27mm"
 			(at 256.54 110.49 0)
 			(hide yes)
@@
 			)
 		)
-		(property "Footprint" ""
+		(property "Footprint" "Package_SO:SOIC-14_3.9x8.7mm_P1.27mm"
 			(at 152.4 68.58 0)
 			(hide yes)
@@
 			)
 		)
-		(property "Footprint" ""
+		(property "Footprint" "Package_SO:SOIC-14_3.9x8.7mm_P1.27mm"
 			(at 124.46 172.72 0)
 			(hide yes)
@@
 			)
 		)
-		(property "Footprint" ""
+		(property "Footprint" "Package_SO:SOIC-14_3.9x8.7mm_P1.27mm"
 			(at 203.2 110.49 0)
 			(hide yes)
@@
 			)
 		)
-		(property "Footprint" ""
+		(property "Footprint" "Package_SO:SOIC-14_3.9x8.7mm_P1.27mm"
 			(at 203.2 68.58 0)
 			(hide yes)
@@
 			)
 		)
-		(property "Footprint" ""
+		(property "Footprint" "Package_SO:SOIC-14_3.9x8.7mm_P1.27mm"
 			(at 307.34 85.09 0)
 			(hide yes)
@@
 			)
 		)
-		(property "Footprint" ""
+		(property "Footprint" "Package_SO:SOIC-14_3.9x8.7mm_P1.27mm"
 			(at 153.67 110.49 0)
 			(hide yes)
