File: fieldRadio_1.2/clock.kicad_sch (KiCad schematic)
At the start: 8 parts, among them J9 Conn_01x02, U8 Si5351A-B-GT, Y2 25MHz

Commit message: updating schematics for fieldRadio_1.2
Parts:
- removed J9: Conn_01x02, Connector_PinHeader_2.54mm:PinHeader_1x02_P2.54mm_Vertical, symbol Connector_Generic:Conn_01x02
- added J19: Conn_01x03, Connector_PinHeader_2.54mm:PinHeader_1x03_P2.54mm_Vertical, symbol Connector_Generic:Conn_01x03
- R135: now fitted
Connections:
- net CLK0: now also J19.1 (Pin_1)
- net CLK1: now also J19.2 (Pin_2)
- net CLK2: now also J19.3 (Pin_3)
Other:
- moved on the sheet: C133, C134, R133, R134, U8, Y2

Commit message: more jlcpcb part number work
Parts:
- C133, C134: value 0.22uF -> 220nF; footprint Capacitor_SMD:C_0603_1608Metric_Pad1.08x0.95mm_HandSolder -> PCM_JLCPCB:C_0603; symbol Device:C_Small -> PCM_JLCPCB-Capacitors:0603,220nF; Attrition Qty (none) -> 10; Capacitance (none) -> 220nF; Category (none) -> Capacitors,Multilayer Ceramic Capacitors MLCC - SMD/SMT; Class (none) -> Basic Component; LCSC (none) -> C21120; Manufacturer (none) -> Samsung Electro-Mechanics; Minimum Qty (none) -> 20; Part (none) -> CL10B224KA8NNNC; Price (none) -> 0.009USD; Process (none) -> SMT; Stock (none) -> 781839; Temperature Coefficient (none) -> X7R; Tolerance (none) -> ±10%; Voltage Rated (none) -> 25V
- R133, R134, R135: value 47 -> 47Ω; footprint Resistor_SMD:R_0603_1608Metric_Pad0.98x0.95mm_HandSolder -> PCM_JLCPCB:R_0603; symbol Device:R_US -> PCM_JLCPCB-Resistors:0603,47Ω; Attrition Qty (none) -> 10; Category (none) -> Resistors,Chip Resistor - Surface Mount; Class (none) -> Basic Component; LCSC (none) -> C23182; Manufacturer (none) -> UNI-ROYAL(Uniroyal Elec); Minimum Qty (none) -> 20; Operating Temperature Range (none) -> -55°C~+155°C; Overload Voltage (Max) (none) -> 75V; Part (none) -> 0603WAF470JT5E; Power(Watts) (none) -> 100mW; Price (none) -> 0.004USD; Process (none) -> SMT; Resistance (none) -> 47Ω; Stock (none) -> 1005542; Temperature Coefficient (none) -> ±100ppm/°C; Tolerance (none) -> ±1%; Type (none) -> Thick Film Resistors
- U8: JLCPCB (none) -> C504891
- Y2: JLCPCB (none) -> C596913
Other:
- moved on the sheet: C133, C134

Commit message: continued symbol property updates
Parts:
- J19: now left out of the parts list
Changed lines of the file:
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@@
 		(body_style 1)
 		(exclude_from_sim no)
-		(in_bom yes)
+		(in_bom no)
 		(on_board yes)
 		(in_pos_files yes)

Commit message: ready to start layout
Parts:
- U8: LCSC (none) -> C504891
- Y2: LCSC (none) -> C596913
Changed lines of the file:
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@@
+			)
+		)
+		(property "LCSC" "C504891"
+			(at 200.66 90.17 0)
+			(hide yes)
+			(show_name no)
+			(do_not_autoplace no)
+			(effects
+				(font
+					(size 1.27 1.27)
+				)
 			)
 		)
@@
 			(at 166.243 85.09 90)
 			(hide yes)
+			(show_name no)
+			(do_not_autoplace no)
+			(effects
+				(font
+					(size 1.27 1.27)
+				)
+			)
+		)
+		(property "LCSC" "C596913"
+			(at 166.243 85.09 90)
+			(hide yes)

Commit message: Starting fieldRadio1.2 layout
Parts:
- renumbered C133 to C164, C134 to C165, J19 to J16, R133 to R146, R134 to R147, R135 to R148, U8 to U26
Changed lines of the file:
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@@
 		(dnp no)
 		(fields_autoplaced yes)
-		(property "Reference" "U8"
+		(property "Reference" "U26"
 			(at 202.9834 102.235 0)
 			(show_name no)
@@
 			(project "fieldRadio_1.2"
 				(path "/a1d1b2b0-2f27-4dc0-94ba-bb0e02933617/07566e3b-8dce-4b8a-bb35-93365cd4b65e"
-					(reference "U8")
+					(reference "U26")
 					(unit 1)
 				)
@@
 		(in_pos_files yes)
 		(dnp no)
-		(property "Reference" "#PWR038"
+		(property "Reference" "#PWR051"
 			(at 200.66 111.76 0)
 			(hide yes)
@@
 			(project "fieldRadio_1.2"
 				(path "/a1d1b2b0-2f27-4dc0-94ba-bb0e02933617/07566e3b-8dce-4b8a-bb35-93365cd4b65e"
-					(reference "#PWR038")
+					(reference "#PWR051")
 					(unit 1)
 				)
@@
 		(in_pos_files yes)
 		(dnp no)
-		(property "Reference" "R135"
+		(property "Reference" "R148"
 			(at 216.535 93.345 90)
 			(show_name no)
@@
 			(project "fieldRadio_1.2"
 				(path "/a1d1b2b0-2f27-4dc0-94ba-bb0e02933617/07566e3b-8dce-4b8a-bb35-93365cd4b65e"
-					(reference "R135")
+					(reference "R148")
 					(unit 1)
 				)
@@
 		(in_pos_files yes)
 		(dnp no)
-		(property "Reference" "#PWR037"
+		(property "Reference" "#PWR050"
 			(at 165.608 96.52 0)
 			(hide yes)
@@
 			(project "fieldRadio_1.2"
 				(path "/a1d1b2b0-2f27-4dc0-94ba-bb0e02933617/07566e3b-8dce-4b8a-bb35-93365cd4b65e"
-					(reference "#PWR037")
+					(reference "#PWR050")
 					(unit 1)
 				)
@@
 		(dnp no)
 		(fields_autoplaced yes)
-		(property "Reference" "J19"
+		(property "Reference" "J16"
 			(at 252.73 73.6599 0)
 			(show_name no)
@@
 			(project "fieldRadio_1.2"
 				(path "/a1d1b2b0-2f27-4dc0-94ba-bb0e02933617/07566e3b-8dce-4b8a-bb35-93365cd4b65e"
-					(reference "J19")
+					(reference "J16")
 					(unit 1)
 				)
@@
 		(in_pos_files yes)
 		(dnp no)
-		(property "Reference" "R133"
+		(property "Reference" "R146"
 			(at 216.535 83.185 90)
 			(show_name no)
@@
 			(project "fieldRadio_1.2"
 				(path "/a1d1b2b0-2f27-4dc0-94ba-bb0e02933617/07566e3b-8dce-4b8a-bb35-93365cd4b65e"
-					(reference "R133")
+					(reference "R146")
 					(unit 1)
 				)
@@
 		(in_pos_files yes)
 		(dnp no)
-		(property "Reference" "C133"
+		(property "Reference" "C164"
 			(at 137.16 78.105 0)
 			(show_name no)
@@
 			(project "fieldRadio_1.2"
 				(path "/a1d1b2b0-2f27-4dc0-94ba-bb0e02933617/07566e3b-8dce-4b8a-bb35-93365cd4b65e"
-					(reference "C133")
+					(reference "C164")
 					(unit 1)
 				)
@@
 		(in_pos_files yes)
 		(dnp no)
-		(property "Reference" "C134"
+		(property "Reference" "C165"
 			(at 146.05 78.105 0)
 			(show_name no)
@@
 			(project "fieldRadio_1.2"
 				(path "/a1d1b2b0-2f27-4dc0-94ba-bb0e02933617/07566e3b-8dce-4b8a-bb35-93365cd4b65e"
-					(reference "C134")
+					(reference "C165")
 					(unit 1)
 				)
@@
 		(in_pos_files yes)
 		(dnp no)
-		(property "Reference" "R134"
+		(property "Reference" "R147"
 			(at 216.535 88.265 90)
 			(show_name no)
@@
 			(project "fieldRadio_1.2"
 				(path "/a1d1b2b0-2f27-4dc0-94ba-bb0e02933617/07566e3b-8dce-4b8a-bb35-93365cd4b65e"
-					(reference "R134")
+					(reference "R147")
 					(unit 1)
 				)
