File: fieldRadio_1.2/controller.kicad_sch (KiCad schematic)
At the start: 85 parts, among them J11 Conn_01x04, J13 Conn_01x02, J14 Conn_01x02, J15 Conn_01x02, J16 Conn_01x02, J17 Conn_01x02, Q19 MOSFET-NCHANNELBSS138, Q23 BSS123, U7 MCP1801-3.3V, Y1 32.768kHz

Commit message: updating schematics for fieldRadio_1.2
Parts:
- removed C113, C115, C116, C118, C119, C123, C124, C125, C126, C127, C128: 0.1uF, Capacitor_SMD:C_0603_1608Metric_Pad1.08x0.95mm_HandSolder, symbol Device:C
- removed J13, J14, J15, J16, J17: Conn_01x02, Connector_PinHeader_2.54mm:PinHeader_1x02_P2.54mm_Vertical, symbol Connector_Generic:Conn_01x02
- removed Q23: BSS123, Package_TO_SOT_SMD:SOT-23-3, symbol Device:Q_NMOS_GSD
- removed R100, R104, R108, R113: 39K, Resistor_SMD:R_0603_1608Metric_Pad0.98x0.95mm_HandSolder, symbol main-eagle-import:RESISTOR0603
- removed R101, R103, R105, R107, R109, R114, R121, R123, R126, R128, R130, R132: 1K, Resistor_SMD:R_0603_1608Metric_Pad0.98x0.95mm_HandSolder, symbol main-eagle-import:RESISTOR0603
- removed R102, R106, R120, R122, R125, R127, R129, R131: 39k, Resistor_SMD:R_0603_1608Metric_Pad0.98x0.95mm_HandSolder, symbol main-eagle-import:RESISTOR0603
- removed R64: 47K, Resistor_SMD:R_0603_1608Metric_Pad0.98x0.95mm_HandSolder, symbol main-eagle-import:RESISTOR0603
Connections:
- net BTN_BAND_SEL: now also U$4.27 (P3.1/UCA1STE)
- net BTN_DIGIT_SEL: now also U$4.25 (P2.3/TA2.0)
- net BTN_FILTER_SEL: now also U$4.26 (P3.4/TA2CLK/COMP0OUT)
- net BTN_MENU: now also U$4.33 (P4.0/TA3.1)
- net BTN_MODE: now also U$4.32 (P3.7/TA3.2)
- net BTN_MUTE: now also U$4.24 (P3.3/TA2.1)
- net BTN_SPOT: now also U$4.29 (P2.5/UCA1RXD/UCA1SOMI)
- net BTN_TXMODE: now also U$4.21 (P5.7/TA2.1/COMP0.2)
- net shiftClk: now reaches U$4.28 (P2.4/UCA1CLK)
- net VDD_AMP_ENABLE: now reaches U$4.23 (P3.0/TA2.2)
- net serData: now reaches U$4.30 (P2.6/UCA1TXD/UCA1SIMO)
- net sel_binaural: now reaches U$4.20 (P5.6/UCB0STE/TA2.0)
- net VDD_DRV_ENABLE: now reaches U$4.4 (P1.4/UCA0TXD/UCA0SIMO/TA1.2/TCK/A4/VREF+)
- net BAND_15M: no longer names the net of U$4.44 (P5.1/UCA0RXD/UCA0SOMI/TB0.3)
- net BAND_17M renamed ~{RF_ENABLE}
- net BAND_20M: no longer names the net of U$4.42 (P4.7/UCA0STE/TB0.1)
- net BAND_30M: no longer names the net of U$4.41 (P6.2/TB0.0)
- net BAND_40M renamed BTN_BIN_MON
- net SIDEBAND_SEL renamed regClk
Other:
- note removed: "PTT"
- moved on the sheet: R93, RV2

Commit message: Working on fieldRadio_1.2 schematics
Parts:
- added C113, C136, C140: 0.1uF, Capacitor_SMD:C_0603_1608Metric_Pad1.08x0.95mm_HandSolder, symbol Device:C
- added R100, R101, R102, R107: 1K, Resistor_SMD:R_0603_1608Metric_Pad0.98x0.95mm_HandSolder, symbol main-eagle-import:RESISTOR0603
- added R103, R104, R105, R106: 39K, Resistor_SMD:R_0603_1608Metric_Pad0.98x0.95mm_HandSolder, symbol main-eagle-import:RESISTOR0603
Connections:
- net BTN_TXMODE: now also R106.1, R107.2; no longer U$4.21 (P5.7/TA2.1/COMP0.2)
- net GND: now also C113.2, C136.2, C140.2
- net VDD3.3: now also R100.1, R101.1, R102.1, R107.1
- net ~{RF_ENABLE}: now also U$4.41 (P6.2/TB0.0); no longer U$4.43 (P5.0/UCA0CLK/TB0.2)
- net at C132.1, U$4.45 (P5.2/UCA0TXD/UCA0SIMO/TB0.4): now also R103.2
- net at U$4.44 (P5.1/UCA0RXD/UCA0SOMI/TB0.3): now also C136.1, R104.2
- net BTN_BAND_SEL: no longer names the net of U$4.27 (P3.1/UCA1STE)
- net BTN_BIN_MON: no longer names the net of U$4.40 (P6.1/TB0CLK)
- net BTN_DIGIT_SEL: no longer names the net of U$4.25 (P2.3/TA2.0)
- net BTN_FILTER_SEL: no longer names the net of U$4.26 (P3.4/TA2CLK/COMP0OUT)
- net BTN_MENU: no longer names the net of U$4.33 (P4.0/TA3.1)
- net BTN_MODE: no longer names the net of U$4.32 (P3.7/TA3.2)
- net BTN_MUTE: no longer names the net of U$4.24 (P3.3/TA2.1)
- net BTN_SPOT: no longer names the net of U$4.29 (P2.5/UCA1RXD/UCA1SOMI)
- net regClk renamed REG_CLK
- net serData renamed SERIAL_DATA
- net shiftClk renamed SERIAL_CLK
- new net: C140.1, R105.2, U$4.43 (P5.0/UCA0CLK/TB0.2)
- new net: C113.1, R106.2, U$4.21 (P5.7/TA2.1/COMP0.2)
- new net BTN_ENCODER_A: R101.2, R104.1
- new net BTN_ENCODER_B: R100.2, R103.1
- new net BTN_ENCODER_SW: R102.2, R105.1

Commit message: adding jlcpcb part numbers to schematics
Parts:
- C105, C107, C109, C110, C111, C112, C113, C117, C129, C130, C131, C132, C136, C140: footprint Capacitor_SMD:C_0603_1608Metric_Pad1.08x0.95mm_HandSolder -> PCM_JLCPCB:C_0603; symbol Device:C -> PCM_JLCPCB-Capacitors:0603,100nF; Attrition Qty (none) -> 10; Capacitance (none) -> 100nF; Category (none) -> Capacitors,Multilayer Ceramic Capacitors MLCC - SMD/SMT; Class (none) -> Basic Component; LCSC (none) -> C14663; Manufacturer (none) -> YAGEO; Minimum Qty (none) -> 20; Part (none) -> CC0603KRX7R9BB104; Price (none) -> 0.006USD; Process (none) -> SMT; Stock (none) -> 70324515; Temperature Coefficient (none) -> X7R; Tolerance (none) -> ±10%; Voltage Rated (none) -> 50V
- C120: footprint Capacitor_SMD:C_0603_1608Metric_Pad1.08x0.95mm_HandSolder -> PCM_JLCPCB:C_0603; symbol Device:C -> PCM_JLCPCB-Capacitors:0603,1nF; Attrition Qty (none) -> 10; Capacitance (none) -> 1nF; Category (none) -> Capacitors,Multilayer Ceramic Capacitors MLCC - SMD/SMT; Class (none) -> Basic Component; LCSC (none) -> C1588; Manufacturer (none) -> Samsung Electro-Mechanics; Minimum Qty (none) -> 20; Part (none) -> CL10B102KB8NNNC; Price (none) -> 0.006USD; Process (none) -> SMT; Stock (none) -> 6068974; Temperature Coefficient (none) -> X7R; Tolerance (none) -> ±10%; Voltage Rated (none) -> 50V
- R100, R101, R102, R107, R116, R118, R124, R90, R95, R97, R99: value 1K -> 1kΩ; footprint Resistor_SMD:R_0603_1608Metric_Pad0.98x0.95mm_HandSolder -> PCM_JLCPCB:R_0603; symbol main-eagle-import:RESISTOR0603 -> PCM_JLCPCB-Resistors:0603,1kΩ; Attrition Qty (none) -> 10; Category (none) -> Resistors,Chip Resistor - Surface Mount; Class (none) -> Basic Component; LCSC (none) -> C21190; Manufacturer (none) -> UNI-ROYAL(Uniroyal Elec); Minimum Qty (none) -> 20; Operating Temperature Range (none) -> -55°C~+155°C; Overload Voltage (Max) (none) -> 75V; Part (none) -> 0603WAF1001T5E; Power(Watts) (none) -> 100mW; Price (none) -> 0.004USD; Process (none) -> SMT; Resistance (none) -> 1kΩ; Stock (none) -> 27538425; Temperature Coefficient (none) -> ±100ppm/°C; Tolerance (none) -> ±1%; Type (none) -> Thick Film Resistors
- R103, R104, R105, R106, R115, R117, R119, R92, R94, R96, R98: footprint Resistor_SMD:R_0603_1608Metric_Pad0.98x0.95mm_HandSolder -> PCM_JLCPCB:R_0603; symbol main-eagle-import:RESISTOR0603 -> PCM_JLCPCB-Resistors:0603,39kΩ; Attrition Qty (none) -> 10; Category (none) -> Resistors,Chip Resistor - Surface Mount; Class (none) -> Basic Component; LCSC (none) -> C23153; Manufacturer (none) -> UNI-ROYAL(Uniroyal Elec); Minimum Qty (none) -> 20; Operating Temperature Range (none) -> -55°C~+155°C; Overload Voltage (Max) (none) -> 75V; Part (none) -> 0603WAF3902T5E; Power(Watts) (none) -> 100mW; Price (none) -> 0.004USD; Process (none) -> SMT; Resistance (none) -> 39kΩ; Stock (none) -> 323259; Temperature Coefficient (none) -> ±100ppm/°C; Tolerance (none) -> ±1%; Type (none) -> Thick Film Resistors
- R112: value 47K -> 47kΩ; footprint Resistor_SMD:R_0603_1608Metric_Pad0.98x0.95mm_HandSolder -> PCM_JLCPCB:R_0603; symbol main-eagle-import:RESISTOR0603 -> PCM_JLCPCB-Resistors:0603,47kΩ; Attrition Qty (none) -> 10; Category (none) -> Resistors,Chip Resistor - Surface Mount; Class (none) -> Basic Component; LCSC (none) -> C25819; Manufacturer (none) -> UNI-ROYAL(Uniroyal Elec); Minimum Qty (none) -> 20; Operating Temperature Range (none) -> -55°C~+155°C; Overload Voltage (Max) (none) -> 75V; Part (none) -> 0603WAF4702T5E; Power(Watts) (none) -> 100mW; Price (none) -> 0.004USD; Process (none) -> SMT; Resistance (none) -> 47kΩ; Stock (none) -> 2267414; Temperature Coefficient (none) -> ±100ppm/°C; Tolerance (none) -> ±1%; Type (none) -> Thick Film Resistors
Connections:
- net BTN_ENCODER_A: no longer R101.2, R104.1
- net BTN_ENCODER_B: no longer R100.2, R103.1
- net BTN_ENCODER_SW: no longer R102.2, R105.1
- net BTN_TXMODE: no longer R106.1, R107.2
- net GND: no longer R90.2, R92.1
- net PADDLE_DAH: no longer R117.2, R118.2
- net PADDLE_DIT: no longer R119.2, R124.2
- net STRAIGHT_KEY: no longer R115.2, R116.2
- net TUNER_ENCODER_A: no longer R96.1, R97.2
- net TUNER_ENCODER_B: no longer R94.1, R95.2
- net TUNER_ENCODER_SW: no longer R98.1, R99.2
- net VDD3.3: no longer R100.1, R101.1, R102.1, R107.1, R112.2, R116.1, R118.1, R124.1, R95.1, R97.1, R99.1
- net at C136.1, U$4.44 (P5.1/UCA0RXD/UCA0SOMI/TB0.3): no longer R104.2
- net at C131.1, U$4.36 (P2.7/UCB1STE): no longer R115.1
- net at C111.1, U$4.17 (P4.5/UCB0SOMI/UCB0SCL/TA3.2): no longer R96.2
- net at C120.2, J11.4 (Pin_4), U$4.2 (RST/NMI/SBWTDIO): no longer R112.1
- net at Q19.1 (G), U$4.22 (P6.0/TA2.2/COMP0.3): no longer R92.2
- net at C140.1, U$4.43 (P5.0/UCA0CLK/TB0.2): no longer R105.2
- net at C112.1, U$4.18 (P4.6/UCB0SIMO/UCB0SDA/TA3.1): no longer R98.2
- net at C130.1, U$4.35 (P4.2/TA3CLK): no longer R117.1
- net at C129.1, U$4.34 (P4.1/TA3.0): no longer R119.1
- net at C105.1, R89.2, U$4.12 (P1.0/UCB0STE/TA0CLK/A0/VEREF+): no longer R90.1
- net at C113.1, U$4.21 (P5.7/TA2.1/COMP0.2): no longer R106.2
- net at C110.1, U$4.16 (P2.2/ACLK/COMP0.1): no longer R94.2
- net at C132.1, U$4.45 (P5.2/UCA0TXD/UCA0SIMO/TB0.4): no longer R103.2

Commit message: more jlcpcb part number work
Parts:
- removed C108: 470pF, Capacitor_SMD:C_0603_1608Metric_Pad1.08x0.95mm_HandSolder, symbol Device:C
- removed U7: MCP1801-3.3V, Package_TO_SOT_SMD:SOT-23-5, symbol Regulator_Linear:MIC5219-3.3YM5
- added C108: 1uF, PCM_JLCPCB:C_0603, symbol PCM_JLCPCB-Capacitors:0603,1uF
- added R108: 1kΩ, PCM_JLCPCB:R_0603, symbol PCM_JLCPCB-Resistors:0603,1kΩ
- added U31: MIC5235-3.3YM5, Package_TO_SOT_SMD:SOT-23-5, symbol Regulator_Linear:MIC5205-3.3YM5
- C106: footprint Capacitor_SMD:C_0603_1608Metric_Pad1.08x0.95mm_HandSolder -> PCM_JLCPCB:C_0603; symbol Device:C -> PCM_JLCPCB-Capacitors:0603,1uF; Attrition Qty (none) -> 10; Capacitance (none) -> 1uF; Category (none) -> Capacitors,Multilayer Ceramic Capacitors MLCC - SMD/SMT; Class (none) -> Basic Component; LCSC (none) -> C15849; Manufacturer (none) -> Samsung Electro-Mechanics; Minimum Qty (none) -> 20; Part (none) -> CL10A105KB8NNNC; Price (none) -> 0.008USD; Process (none) -> SMT; Stock (none) -> 11535980; Temperature Coefficient (none) -> X5R; Tolerance (none) -> ±10%; Voltage Rated (none) -> 50V
- C114: footprint Capacitor_THT:CP_Radial_D5.0mm_P2.00mm -> PCM_JLCPCB:C_0805; symbol Device:C_Polarized -> PCM_JLCPCB-Capacitors:0805,10uF; Attrition Qty (none) -> 10; Capacitance (none) -> 10uF; Category (none) -> Capacitors,Multilayer Ceramic Capacitors MLCC - SMD/SMT; Class (none) -> Basic Component; LCSC (none) -> C15850; Manufacturer (none) -> Samsung Electro-Mechanics; Minimum Qty (none) -> 20; Part (none) -> CL21A106KAYNNNE; Price (none) -> 0.014USD; Process (none) -> SMT; Stock (none) -> 6525809; Temperature Coefficient (none) -> X5R; Tolerance (none) -> ±10%; Voltage Rated (none) -> 25V
- Q19: value MOSFET-NCHANNELBSS138 -> BSS138; footprint Package_TO_SOT_SMD:SOT-23 -> PCM_JLCPCB:Q_SOT-23; symbol main-eagle-import:MOSFET-NCHANNELBSS138 -> PCM_JLCPCB-Transistors:NMOS,BSS138; Attrition Qty (none) -> 5; Category (none) -> Triode/MOS Tube/Transistor,MOSFETs; Class (none) -> Preferred Component; Continuous Drain Current (Id) (none) -> 340mA; Drain Source On Resistance (RDS(on)@Vgs,Id) (none) -> 2.5Ω@10V,0.34A; Drain Source Voltage (Vdss) (none) -> null; Gate Threshold Voltage (Vgs(th)@Id) (none) -> 1.6V@250uA; Input Capacitance (Ciss@Vds) (none) -> 17.5pF@25V; LCSC (none) -> C7420339; Manufacturer (none) -> hongjiacheng; Minimum Qty (none) -> 10; Operating Temperature (none) -> -55°C~+150°C; Part (none) -> BSS138; Power Dissipation (Pd) (none) -> 350mW; Price (none) -> 0.021USD; Process (none) -> SMT; Reverse Transfer Capacitance (Crss@Vds) (none) -> 6.5pF@25V; Stock (none) -> 257620; Total Gate Charge (Qg@Vgs) (none) -> 1.7nC@10V; Type (none) -> null
- R110, R111: value 2.7K -> 2.7kΩ; footprint Resistor_SMD:R_0603_1608Metric_Pad0.98x0.95mm_HandSolder -> PCM_JLCPCB:R_0603; symbol main-eagle-import:RESISTOR0603 -> PCM_JLCPCB-Resistors:0603,2.7kΩ; Attrition Qty (none) -> 10; Category (none) -> Resistors,Chip Resistor - Surface Mount; Class (none) -> Basic Component; LCSC (none) -> C13167; Manufacturer (none) -> UNI-ROYAL(Uniroyal Elec); Minimum Qty (none) -> 20; Operating Temperature Range (none) -> -55°C~+155°C; Overload Voltage (Max) (none) -> 75V; Part (none) -> 0603WAF2701T5E; Power(Watts) (none) -> 100mW; Price (none) -> 0.004USD; Process (none) -> SMT; Resistance (none) -> 2.7kΩ; Stock (none) -> 1077645; Temperature Coefficient (none) -> ±100ppm/°C; Tolerance (none) -> ±1%; Type (none) -> Thick Film Resistors
- R89: value 9.09K -> 9.1kΩ; footprint Resistor_SMD:R_0603_1608Metric_Pad0.98x0.95mm_HandSolder -> PCM_JLCPCB:R_0603; symbol main-eagle-import:RESISTOR0603 -> PCM_JLCPCB-Resistors:0603,9.1kΩ; Attrition Qty (none) -> 10; Category (none) -> Resistors,Chip Resistor - Surface Mount; Class (none) -> Basic Component; LCSC (none) -> C23260; Manufacturer (none) -> UNI-ROYAL(Uniroyal Elec); Minimum Qty (none) -> 20; Operating Temperature Range (none) -> -55°C~+155°C; Overload Voltage (Max) (none) -> 75V; Part (none) -> 0603WAF9101T5E; Power(Watts) (none) -> 100mW; Price (none) -> 0.004USD; Process (none) -> SMT; Resistance (none) -> 9.1kΩ; Stock (none) -> 391306; Temperature Coefficient (none) -> ±100ppm/°C; Tolerance (none) -> ±1%; Type (none) -> Thick Film Resistors
- R91: value 330 -> 330Ω; footprint Resistor_SMD:R_0603_1608Metric_Pad0.98x0.95mm_HandSolder -> PCM_JLCPCB:R_0603; symbol main-eagle-import:RESISTOR0603 -> PCM_JLCPCB-Resistors:0603,330Ω; Attrition Qty (none) -> 10; Category (none) -> Resistors,Chip Resistor - Surface Mount; Class (none) -> Basic Component; LCSC (none) -> C23138; Manufacturer (none) -> UNI-ROYAL(Uniroyal Elec); Minimum Qty (none) -> 20; Operating Temperature Range (none) -> -55°C~+155°C; Overload Voltage (Max) (none) -> 75V; Part (none) -> 0603WAF3300T5E; Power(Watts) (none) -> 100mW; Price (none) -> 0.004USD; Process (none) -> SMT; Resistance (none) -> 330Ω; Stock (none) -> 2977706; Temperature Coefficient (none) -> ±100ppm/°C; Tolerance (none) -> ±1%; Type (none) -> Thick Film Resistors
- R93: value 100 -> 100Ω; footprint Resistor_SMD:R_0603_1608Metric_Pad0.98x0.95mm_HandSolder -> PCM_JLCPCB:R_0603; symbol main-eagle-import:RESISTOR0603 -> PCM_JLCPCB-Resistors:0603,100Ω; Attrition Qty (none) -> 10; Category (none) -> Resistors,Chip Resistor - Surface Mount; Class (none) -> Basic Component; LCSC (none) -> C22775; Manufacturer (none) -> UNI-ROYAL(Uniroyal Elec); Minimum Qty (none) -> 20; Operating Temperature Range (none) -> -55°C~+155°C; Overload Voltage (Max) (none) -> 75V; Part (none) -> 0603WAF1000T5E; Power(Watts) (none) -> 100mW; Price (none) -> 0.004USD; Process (none) -> SMT; Resistance (none) -> 100Ω; Stock (none) -> 8202320; Temperature Coefficient (none) -> ±200ppm/°C; Tolerance (none) -> ±1%; Type (none) -> Thick Film Resistors
- U$4: JLCPCB (none) -> C1340815
- Y1: JLCPCB (none) -> C510776
Connections:
- net BTN_ENCODER_A: now also R101.2, R104.2
- net BTN_ENCODER_B: now also R100.2, R103.2
- net BTN_ENCODER_SW: now also R102.2, R105.2
- net BTN_TXMODE: now also R106.1, R107.1
- net GND: now also R90.2, R92.2, C108.2, U31.2 (GND)
- net LCD_A: now also R93.1; no longer R93.2
- net PADDLE_DAH: now also R117.2, R118.1
- net PADDLE_DIT: now also R119.2, R124.1
- net STRAIGHT_KEY: now also R115.2, R116.1
- net TUNER_ENCODER_A: now also R96.1, R97.1
- net TUNER_ENCODER_B: now also R94.1, R95.1
- net TUNER_ENCODER_SW: now also R98.1, R99.1
- net TX_LED: now also R91.1; no longer R91.2
- net VDD3.3: now also R100.1, R101.1, R102.1, R107.2, R112.2, R116.2, R118.2, R124.2, R95.2, R97.2, R99.2, C108.1, U31.5 (OUT)
- net VDD5: now also R93.2, R108.1, U31.1 (IN); no longer R93.1
- net at C136.1, U$4.44 (P5.1/UCA0RXD/UCA0SOMI/TB0.3): now also R104.1
- net at R115.1: now also C131.1, U$4.36 (P2.7/UCB1STE)
- net at R96.2: now also C111.1, U$4.17 (P4.5/UCB0SOMI/UCB0SCL/TA3.2)
- net at R112.1: now also C120.2, J11.4 (Pin_4), U$4.2 (RST/NMI/SBWTDIO)
- net at R92.1: now also Q19.1 (G), U$4.22 (P6.0/TA2.2/COMP0.3)
- net at C140.1, U$4.43 (P5.0/UCA0CLK/TB0.2): now also R105.1
- net at C112.1, U$4.18 (P4.6/UCB0SIMO/UCB0SDA/TA3.1): now also R98.2
- net at C130.1, U$4.35 (P4.2/TA3CLK): now also R117.1
- net at Q19.3 (D): now also R91.2; no longer R91.1
- net at R119.1: now also C129.1, U$4.34 (P4.1/TA3.0)
- net at R90.1: now also C105.1, R89.2, U$4.12 (P1.0/UCB0STE/TA0CLK/A0/VEREF+)
- net at C113.1, U$4.21 (P5.7/TA2.1/COMP0.2): now also R106.2
- net at C110.1, U$4.16 (P2.2/ACLK/COMP0.1): now also R94.2
- net at C132.1, U$4.45 (P5.2/UCA0TXD/UCA0SIMO/TB0.4): now also R103.1
- new net: R108.2, U31.3 (EN)
Other:
- moved on the sheet: R100, R101, R102, R103, R104, R105, R106, R107, R112, R115, R116, R117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

Commit message: continued symbol property updates
Parts:
- C105, C107, C109, C110, C111, C112, C113, C117, C129, C130, C131, C132, C136, C140: JLCPCB (none) -> C14663
- C106, C108: JLCPCB (none) -> C15849
- C114: JLCPCB (none) -> C15850
- C120: JLCPCB (none) -> C1588
- C121, C122: footprint Capacitor_SMD:C_0603_1608Metric_Pad1.08x0.95mm_HandSolder -> PCM_JLCPCB:C_0603; symbol Device:C -> PCM_JLCPCB-Capacitors:0603,22pF; Attrition Qty (none) -> 10; Capacitance (none) -> 22pF; Category (none) -> Capacitors,Multilayer Ceramic Capacitors MLCC - SMD/SMT; Class (none) -> Basic Component; JLCPCB (none) -> C1653; LCSC (none) -> C1653; Manufacturer (none) -> Samsung Electro-Mechanics; Minimum Qty (none) -> 20; Part (none) -> CL10C220JB8NNNC; Price (none) -> 0.007USD; Process (none) -> SMT; Stock (none) -> 1531147; Temperature Coefficient (none) -> C0G; Tolerance (none) -> ±5%; Voltage Rated (none) -> 50V
- J11, RV2: now left out of the parts list
- Q19: JLCPCB (none) -> C7420339
- R100, R101, R102, R107, R108, R116, R118, R124, R90, R95, R97, R99: JLCPCB (none) -> C21190
- R103, R104, R105, R106, R115, R117, R119, R92, R94, R96, R98: JLCPCB (none) -> C23153
- R110, R111: JLCPCB (none) -> C13167
- R112: JLCPCB (none) -> C25819
- R89: JLCPCB (none) -> C23260
- R91: JLCPCB (none) -> C23138
- R93: JLCPCB (none) -> C22775
- U31: JLCPCB (none) -> C7202997

Commit message: ready to start layout
Parts:
- added C151, C153, C155: 0.1uF, PCM_JLCPCB:C_0603, symbol PCM_JLCPCB-Capacitors:0603,100nF
- added R114, R120, R121: 39K, PCM_JLCPCB:R_0603, symbol PCM_JLCPCB-Resistors:0603,39kΩ
- added R122, R123, R125: 1kΩ, PCM_JLCPCB:R_0603, symbol PCM_JLCPCB-Resistors:0603,1kΩ
- U$4: LCSC (none) -> C1340815
- Y1: LCSC (none) -> C510776
Connections:
- net GND: now also C151.2, C153.2, C155.2
- net VDD3.3: now also R122.1, R123.1, R125.1
- net ~{RF_ENABLE}: now also U$4.33 (P4.0/TA3.1); no longer U$4.41 (P6.2/TB0.0)
- net VDD_SNS: now reaches C105.1, R89.2, R90.1, U$4.12 (P1.0/UCB0STE/TA0CLK/A0/VEREF+)
- net LCD_DB3: now reaches U$4.24 (P3.3/TA2.1)
- net LCD_DB2: now reaches U$4.25 (P2.3/TA2.0)
- net LCD_DB1: now reaches U$4.26 (P3.4/TA2CLK/COMP0OUT)
- net LCD_DB0: now reaches U$4.27 (P3.1/UCA1STE)
- net at U$4.40 (P6.1/TB0CLK): now also C155.1, R121.1
- net at U$4.42 (P4.7/UCA0STE/TB0.1): now also C151.1, R114.1
- net BTN_ENCODER_A renamed LED_ENCODER_A
- net BTN_ENCODER_B renamed LED_ENCODER_B
- net BTN_ENCODER_SW renamed LED_ENCODER_SW
- new net: C153.1, R120.1, U$4.41 (P6.2/TB0.0)
- new net MEN_ENCODER_A: R114.2, R122.2
- new net MEN_ENCODER_B: R120.2, R123.2
- new net MEN_ENCODER_SW: R121.2, R125.2
Other:
- moved on the sheet: C129, C130, C131
