File: fieldRadio_1.2/fieldRadio_1.2.kicad_pcb (KiCad board)
At the start: 4 copper layers, 159 x 159 mm, 486 parts, among them IC1 SN74CBTLV3253, J1 Conn_01x02, J10 Conn_01x04, J11 Conn_01x16, J12 Conn_01x03, J13 Conn_01x02, J14 Conn_01x04, J15 Conn_01x08, J16 Conn_01x03, J17 Conn_01x03, J18 Conn_01x03, J2 Conn_01x02, J3 Conn_01x03, J4 Conn_01x14, J5 AudioJack2_Switch, J6 AudioJack3_Switch, J7 Conn_01x02, J8 Conn_01x04, J9 AudioJack3_Switch, K1 G6SU-2, K2 G6SU-2, K3 G6SU-2, K4 G6SU-2, K5 G6SU-2, K6 G6SU-2, Q1 MMBT3904, Q10 BSS138, Q11 IRF9540, Q2 MMBT3904, Q3 PMV240SP, Q4 MMBT3904, Q5 PMV240SP, Q6 DMN10H220LPDW, Q7 BC847BS, Q8 PMV240SP, Q9 J309, SW1 SW_Slide_DPDT, T1 T50-TRIFILAR, U1 OPA1679, U10 MIC5235-3.3YM5, U11 LMR51430, U12 UCC27517DBVR, U13 UCC27517DBVR, U14 LMR51430, U15 OPA1679, U16 OPA1679, U17 TS5A3159ADCK, U18 LMC567, U19 TS5A3159ADCK, U2 OPA1678, U20 TS5A3159ADCK, U21 OPA1679, U22 TS5A3159ADCK, U23 LM4810, U24 MIC5235-3.3YM5, U25 MIC5235-3.3YM5, U26 Si5351A-B-GT, U27 LM1086-5.0, U28 LMR51430, U29 OPA1679, U3 TS5A3159ADCK, U30 OPA1678, U31 TS5A3159ADCK, U32 INA821xD, U33 INA821xD, U4 74HCT595, U5 74ACT125, U6 74ACT244, U7 TLV61047DDC, U8 OPA1678, U9 74LVC2G125, Y1 32.768kHz, Y2 25MHz

Commit message: audio placement first pass completed
Parts:
- moved C97 101.9 mm to (184.8, 168.2)
- moved C89 99.2 mm to (182.0, 176.0), turned to 180 degrees
- moved C90 96.3 mm to (184.8, 179.5), turned to -90 degrees
- moved C91 95.2 mm to (188.2, 168.2), turned to 180 degrees
- moved R61 94.8 mm to (177.0, 171.0), turned to 90 degrees
- moved C96 94.0 mm to (190.8, 179.2), turned to -90 degrees
- moved R68 92.4 mm to (182.5, 174.0)
- moved R66 92.3 mm to (182.5, 170.0)
- moved R65 91.6 mm to (182.5, 171.8)
- moved U17 91.4 mm to (202.2, 161.0)
- moved C87 89.5 mm to (199.8, 174.0), turned to 180 degrees
- moved R58 87.7 mm to (182.0, 178.5), turned to 180 degrees
- moved C95 84.8 mm to (206.5, 167.0)
- moved R53 84.3 mm to (182.0, 180.5)
- moved R52 82.7 mm to (183.2, 182.5)
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
Commit message: placement complete for qsd+audio
Parts:
- moved JP4 226.2 mm to (181.2, 211.2), turned to 90 degrees
- moved R106 215.5 mm to (185.8, 193.2), turned to -90 degrees
- moved R99 212.6 mm to (187.0, 207.8), turned to 90 degrees
- moved Q9 212.1 mm to (190.2, 208.0), turned to -90 degrees
- moved R100 208.9 mm to (191.0, 211.8), turned to 90 degrees
- moved C137 208.7 mm to (184.8, 188.2)
- moved R105 208.2 mm to (193.2, 193.2), turned to -90 degrees
- moved C126 206.8 mm to (185.2, 207.8), turned to -90 degrees
- moved C127 205.3 mm to (187.0, 211.0), turned to 90 degrees
- moved U32 204.0 mm to (189.5, 190.8), turned to 90 degrees
- moved R101 202.6 mm to (197.5, 214.2), turned to 180 degrees
- moved C138 200.8 mm to (192.5, 186.0)
- moved R107 199.1 mm to (202.0, 193.2), turned to -90 degrees
- moved U24 196.5 mm to (205.8, 200.6), turned to 180 degrees
- moved R103 195.0 mm to (203.8, 210.0), turned to -90 degrees
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
Commit message: continued placement work
Parts:
- removed C167, C169: 4.7uF, PCM_JLCPCB:C_0805
- removed C170, C173: 100nF, PCM_JLCPCB:C_0603
- removed C174, C175: 22uF, PCM_JLCPCB:C_0805
- removed C176: 100uF, Capacitor_SMD:C_Elec_6.3x5.8
- removed J17, J18: Conn_01x03, Connector_Wire:SolderWire-0.75sqmm_1x03_P4.8mm_D1.25mm_OD2.3mm
- removed L25: 6.8uH, Inductor_SMD:L_TechFuse_SL0624
- removed R149: 10kΩ, PCM_JLCPCB:R_0603
- removed R150: 12kΩ, PCM_JLCPCB:R_0603
- removed R151: 2kΩ, PCM_JLCPCB:R_0603
- removed R152: 100k, PCM_JLCPCB:R_0603
- removed U28: LMR51430, Package_TO_SOT_SMD:SOT-23-6
- U27: value LM1086-5.0 -> L7805ABD2T-TR; footprint Package_TO_SOT_THT:TO-220-3_Vertical -> Package_TO_SOT_SMD:TO-263-2
- moved Q7 439.5 mm to (-55.8, 125.5)
- moved R49 439.2 mm to (-57.8, 131.2), turned to -90 degrees
- moved R47 438.7 mm to (-56.8, 133.8), turned to 180 degrees
- moved R48 438.2 mm to (-56.8, 129.0)
- moved R50 437.3 mm to (-56.0, 131.2), turned to -90 degrees
- moved R46 436.8 mm to (-55.5, 123.2)
- moved J12 434.8 mm to (-50.0, 116.2)
- moved R41 432.7 mm to (-56.0, 100.5)
- moved C73 431.1 mm to (-61.2, 100.5)
- moved C75 426.4 mm to (-50.0, 124.5), turned to 180 degrees
- moved C77 426.3 mm to (-50.0, 126.8), turned to 180 degrees
- moved U14 425.1 mm to (-50.8, 131.5), turned to 180 degrees
- moved R43 424.1 mm to (-47.5, 98.2)
- moved R44 424.1 mm to (-47.5, 100.5)
- moved R45 424.1 mm to (-47.5, 102.8)
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Connections:
- C166 pad 1: Net-(J17-Pin_3) -> VDD12
- C168 pad 1: Net-(J17-Pin_3) -> VDD12
- C171 pad 1: /powerInput/+5V_Linear -> VDD5
- C172 pad 1: /powerInput/+5V_Linear -> VDD5
- U27 pad 1: GND -> VDD12
- U27 pad 2: /powerInput/+5V_Linear -> GND
- U27 pad 3: Net-(J17-Pin_3) -> VDD5
