File: swrPowerMeter/swrPowerMeter.kicad_pcb (KiCad board)
At the start: 2 copper layers, 60 x 50 mm, 25 parts, among them J3 Conn_01x02, J4 Conn_01x02, J5 Conn_01x02, J6 Conn_Coaxial, J7 Conn_Coaxial

Commit message: taped out
Parts:
- added TP1: TestPoint, TestPoint:TestPoint_THTPad_D2.0mm_Drill1.0mm, F.Cu at (150.2, 104.8)
- added TP2: TestPoint, TestPoint:TestPoint_THTPad_D2.0mm_Drill1.0mm, F.Cu at (162.1, 95.8)
- added TP3: TestPoint, TestPoint:TestPoint_THTPad_D2.0mm_Drill1.0mm, F.Cu at (174.0, 95.8)
- added TP4: TestPoint, TestPoint:TestPoint_THTPad_D2.0mm_Drill1.0mm, F.Cu at (185.9, 95.2)
- C1, C2, C4, C5: footprint PCM_JLCPCB:C_0603 -> Capacitor_SMD:C_0603_1608Metric_Pad1.08x0.95mm_HandSolder
- C3, C6: footprint PCM_JLCPCB:C_0805 -> Capacitor_SMD:C_0805_2012Metric_Pad1.18x1.45mm_HandSolder
- R1, R10, R2, R3, R4, R5, R6, R7, R8, R9: footprint PCM_JLCPCB:R_0603 -> Resistor_SMD:R_0603_1608Metric_Pad0.98x0.95mm_HandSolder
- moved R2 0.28 mm to (165.1, 119.8)
- moved R4 0.12 mm to (173.6, 119.5)
Routing:
- net GND: vias 52 -> 46
Other:
- board size 60 x 50 mm -> 60 x 45.8 mm
